File: coolerpcb.kicad_sch (KiCad schematic)
At the start: 0 parts

Commit message: TMP PCB
Parts:
- added C1: 0.1uF, coolerpcb:0603-NO, symbol coolerpcb-eagle-import:CAP_CERAMIC0603_NO
- added C2: 10uF, coolerpcb:0805-NO, symbol coolerpcb-eagle-import:CAP_CERAMIC0805-NOOUTLINE
- added CONN3, CONN4: STEMMA_I2C_QT, coolerpcb:JST_SH4, symbol coolerpcb-eagle-import:STEMMA_I2C_QT
- added D1: GREEN, coolerpcb:CHIPLED_0603_NOOUTLINE, symbol coolerpcb-eagle-import:LED0603_NOOUTLINE
- added FID3, FID4: FIDUCIAL_1MM, coolerpcb:FIDUCIAL_1MM, symbol coolerpcb-eagle-import:FIDUCIAL_1MM
- added J1: Conn_01x04_Socket, Connector_JST:JST_XH_B4B-XH-A_1x04_P2.50mm_Vertical, symbol Connector:Conn_01x04_Socket
- added JP1: HEADER-1X670MIL, coolerpcb:1X06_ROUND_70, symbol coolerpcb-eagle-import:HEADER-1X670MIL
- added R1: RESISTOR_0603_NOOUT, coolerpcb:0603-NO, symbol coolerpcb-eagle-import:RESISTOR_0603_NOOUT
- added R3: 10K, coolerpcb:RESPACK_4X0603, symbol coolerpcb-eagle-import:RESISTOR_4PACK
- added SJ1: SOLDERJUMPER, coolerpcb:SOLDERJUMPER_ARROW_NOPASTE, symbol coolerpcb-eagle-import:SOLDERJUMPER
- added U$1, U$17, U$19, U$21: MOUNTINGHOLE2.5, coolerpcb:MOUNTINGHOLE_2.5_PLATED, symbol coolerpcb-eagle-import:MOUNTINGHOLE2.5
- added U1: TMP117xxDRV, Package_SON:WSON-6-1EP_2x2mm_P0.65mm_EP1x1.6mm, symbol Sensor_Temperature:TMP117xxDRV
- added X1: TMP117_WSON, coolerpcb:WSON-6, symbol coolerpcb-eagle-import:TMP117_WSON
Connections:
- new net: J1.3 (Pin_3), U1.6 (SDA)
- new net: J1.4 (Pin_4), U1.1 (SCL)
- new net: D1.A, R1.1
- new net ADDR: JP1.6, R3.8 (2), SJ1.1, X1.4 (ADDR)
- new net GND: C1.2, C2.2, CONN3.1 (GND), CONN3.MT1 (MT), CONN3.MT2 (MT), CONN4.1 (GND), CONN4.MT1 (MT), CONN4.MT2 (MT), D1.C, J1.1 (Pin_1), JP1.2, R3.1, U1.2 (GND), U1.3 (ALERT), U1.4 (ADD0), X1.2 (VSS)
- new net INT: JP1.5, R3.7 (2), X1.3 (ALERT)
- new net SCL: CONN3.4 (SCL), CONN4.4 (SCL), JP1.3, R3.4 (1), X1.1 (SCL)
- new net SDA: CONN3.3 (SDA), CONN4.3 (SDA), JP1.4, R3.3 (1), X1.6 (SDA)
- new net VCC: C1.1, C2.1, CONN3.2 (V+), CONN4.2 (V+), J1.2 (Pin_2), JP1.1, R1.2, R3.2 (1), R3.5 (2), R3.6 (2), SJ1.2, U1.5 (V+), X1.5 (VDD)
Other:
- note added: "I2C Pullups & Shift"
- note added: "ON LED"
- note added: "Power supply"
- note added: "STEMMA/I2C Headers"

Commit message: 2/4
Parts:
- removed J1: Conn_01x04_Socket, Connector_JST:JST_XH_B4B-XH-A_1x04_P2.50mm_Vertical, symbol Connector:Conn_01x04_Socket
- added J1: S4B-PH-SM4-TB, S4B_PH_SM4_TB:JST_S4B-PH-SM4-TB, symbol S4B-PH-SM4-TB:S4B-PH-SM4-TB
Connections:
- net GND: now also J1.4
- net VCC: now also J1.3
- net at U1.6 (SDA): now also J1.2
- net at U1.1 (SCL): now also J1.1
Changed lines of the file:
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@@
+	)
+	(symbol
+		(lib_id "S4B-PH-SM4-TB:S4B-PH-SM4-TB")
+		(at 152.4 93.98 90)
+		(unit 1)
+		(exclude_from_sim no)
+		(in_bom yes)
+		(on_board yes)
+		(dnp no)
+		(fields_autoplaced yes)
+		(property "Reference" "J1"
+			(at 161.29 92.0749 90)
+			(effects
+				(font
+					(size 1.27 1.27)
+				)
+				(justify right)
+			)
+		)
+		(property "Value" "S4B-PH-SM4-TB"
+			(at 161.29 94.6149 90)
+			(effects
+				(font
+					(size 1.27 1.27)
+				)
+				(justify right)
+			)
+		)
+		(property "Footprint" "S4B_PH_SM4_TB:JST_S4B-PH-SM4-TB"
+			(at 152.4 93.98 0)
+			(effects
+				(font
+					(size 1.27 1.27)
+				)
+				(justify bottom)
+				(hide yes)
+			)
+		)
+		(property "Datasheet" ""
+			(at 152.4 93.98 0)
+			(effects
+				(font
+					(size 1.27 1.27)
+				)
+				(hide yes)
+			)
+		)
+		(property "Description" ""
+			(at 152.4 93.98 0)
+			(effects
+				(font
+					(size 1.27 1.27)
+				)
+				(hide yes)
+			)
+		)
+		(property "VERIFIER" ""
+			(at 152.4 93.98 0)
+			(effects
+				(font
+					(size 1.27 1.27)
+				)
+				(justify bottom)
+				(hide yes)
+			)
+		)
+		(property "MANUFACTURER" "JST Sales"
+			(at 152.4 93.98 0)
+			(effects
+				(font
+					(size 1.27 1.27)
+				)
+				(justify bottom)
+				(hide yes)
+			)
+		)
+		(property "STANDARD" "Manufacturer Recommendations"
+			(at 152.4 93.98 0)
+			(effects
+				(font
+					(size 1.27 1.27)
+				)
+				(justify bottom)
+				(hide yes)
+			)
+		)
+		(property "MAXIMUM_PACKAGE_HEIGHT" "5.5mm"
+			(at 152.4 93.98 0)
+			(effects
+				(font
+					(size 1.27 1.27)
+				)
+				(justify bottom)
+				(hide yes)
+			)
+		)
+		(property "CREATOR" "DIZAR"
+			(at 152.4 93.98 0)
+			(effects
+				(font
+					(size 1.27 1.27)
+				)
+				(justify bottom)
+				(hide yes)
+			)
+		)
+		(pin "2"
+		)
+		(pin "4"
+		)
+		(pin "1"
+		)
+		(pin "3"
+		)
+		(instances
+			(project ""
+				(path "/3fbae0b3-3e6a-4fc3-bce7-3e63a917950e"
+					(reference "J1")
+					(unit 1)
+				)
+			)
+		)
 	)
 	(symbol
@@
 				)
 			)
-		)
-	)
-	(symbol
-		(lib_id "Connector:Conn_01x04_Socket")
-		(at 154.94 96.52 270)
-		(mirror x)
-		(unit 1)
-		(exclude_from_sim no)
-		(in_bom yes)
-		(on_board yes)
-		(dnp no)
-		(property "Reference" "J1"
-			(at 154.94 93.726 0)
-			(effects
-				(font
-					(size 1.27 1.27)
-				)
-				(justify left)
-			)
-		)
-		(property "Value" "Conn_01x04_Socket"
-			(at 152.654 93.218 0)
-			(effects
-				(font
-					(size 1.27 1.27)
-				)
-				(justify left)
-			)
-		)
-		(property "Footprint" "Connector_JST:JST_XH_B4B-XH-A_1x04_P2.50mm_Vertical"
-			(at 161.544 79.502 0)
-			(effects
-				(font
-					(size 1.27 1.27)
-				)
-				(hide yes)
-			)
-		)
-		(property "Datasheet" "~"
-			(at 154.94 96.52 0)
-			(effects
-				(font
-					(size 1.27 1.27)
-				)
-				(hide yes)
-			)
-		)
-		(property "Description" "Generic connector, single row, 01x04, script generated"
-			(at 154.94 96.52 0)
-			(effects
-				(font
-					(size 1.27 1.27)
-				)
-				(hide yes)
-			)
-		)
-		(pin "1"
-		)
-		(pin "2"
-		)
-		(pin "3"
-		)
-		(pin "4"
-		)
-		(instances
-			(project ""
-				(path "/3fbae0b3-3e6a-4fc3-bce7-3e63a917950e"
-					(reference "J1")
-					(unit 1)
-				)
-			)

Commit message: TMP
Parts:
- removed C1: 0.1uF, coolerpcb:0603-NO, symbol coolerpcb-eagle-import:CAP_CERAMIC0603_NO
- removed C2: 10uF, coolerpcb:0805-NO, symbol coolerpcb-eagle-import:CAP_CERAMIC0805-NOOUTLINE
- removed CONN3, CONN4: STEMMA_I2C_QT, coolerpcb:JST_SH4, symbol coolerpcb-eagle-import:STEMMA_I2C_QT
- removed D1: GREEN, coolerpcb:CHIPLED_0603_NOOUTLINE, symbol coolerpcb-eagle-import:LED0603_NOOUTLINE
- removed JP1: HEADER-1X670MIL, coolerpcb:1X06_ROUND_70, symbol coolerpcb-eagle-import:HEADER-1X670MIL
- removed R1: RESISTOR_0603_NOOUT, coolerpcb:0603-NO, symbol coolerpcb-eagle-import:RESISTOR_0603_NOOUT
- removed R3: 10K, coolerpcb:RESPACK_4X0603, symbol coolerpcb-eagle-import:RESISTOR_4PACK
- removed SJ1: SOLDERJUMPER, coolerpcb:SOLDERJUMPER_ARROW_NOPASTE, symbol coolerpcb-eagle-import:SOLDERJUMPER
- removed X1: TMP117_WSON, coolerpcb:WSON-6, symbol coolerpcb-eagle-import:TMP117_WSON
Other:
- note removed: "I2C Pullups & Shift"
- note removed: "ON LED"
- note removed: "Power supply"
- note removed: "STEMMA/I2C Headers"
- moved on the sheet: J1, U1
