File: RATS117/RATS117.kicad_pcb (KiCad board)
At the start: 2 copper layers, 15 x 13.5 mm, 3 parts, among them J1 S4B-PH-SM4-TB, U1 TMP117xxDRV

Commit message: a
Parts:
- added C1: 0.1uF, Capacitor_SMD:C_1206_3216Metric, B.Cu at (155.5, 93.5)
- moved G*** 1.00 mm to (155.0, 103.0)
Routing:
- net VCC: track 14.8 -> 29.0 mm
- net GND: track 19.6 -> 29.1 mm
Other:
- board size 15 x 13.5 mm -> 17.5 x 15 mm

Commit message: 2/9/26
Parts:
- added JP1: SolderJumper_2_Open, Jumper:SolderJumper-2_P1.3mm_Open_TrianglePad1.0x1.5mm, B.Cu at (155.7, 93.0)
- added JP2: SolderJumper_2_Open, Jumper:SolderJumper-2_P1.3mm_Open_TrianglePad1.0x1.5mm, B.Cu at (143.8, 93.0)
- added R1: 47k, Resistor_SMD:R_1206_3216Metric, B.Cu at (148.0, 91.0)
- moved G*** 11.1 mm to (144.5, 99.5)
- moved C1 4.75 mm to (151.5, 91.0), turned to 90 degrees
Connections:
- U1 pad 4: GND -> Net-(JP1-B)
Routing:
- net Net-(JP1-B): track 0.00 -> 25.0 mm, vias 0 -> 1
- net Net-(JP2-B): track 10.9 -> 24.7 mm
- net VCC: track 29.0 -> 36.1 mm
- net GND: track 29.1 -> 23.7 mm
Other:
- board size 17.5 x 15 mm -> 17.5 x 18.5 mm

Commit message: TMP
Parts:
- moved JP1 1.92 mm to (155.0, 91.2), turned to -90 degrees
- moved JP2 1.92 mm to (144.5, 91.2), turned to -90 degrees
- moved R1 1.04 mm to (148.0, 92.0)
- moved C1 1.00 mm to (151.5, 92.0)
Routing:
- net VCC: track 36.1 -> 11.6 mm, vias 1 -> 0
- net Net-(JP2-B): track 24.7 -> 2.51 mm
- net GND: track 23.7 -> 1.75 mm, vias 1 -> 0
- net Net-(JP1-B): track 25.0 -> 3.52 mm, vias 1 -> 0
- net Net-(U1-SCL): track 19.1 -> 0.00 mm, vias 1 -> 0
- added copper zone on B.Cu, net GND
