File: MainPCB/MAIN_PCB.kicad_sch (KiCad schematic)
At the start: 7 parts

Commit message: c
Parts:
- added J1, J2, J3: S4B-PH-SM4-TB, S4B-PH-SM4-TB:JST_S4B-PH-SM4-TB, symbol S4B-PH-SM4-TB:S4B-PH-SM4-TB
- added U1: DRV8871DDA, Package_SO:Texas_HTSOP-8-1EP_3.9x4.9mm_P1.27mm_EP2.95x4.9mm_Mask2.4x3.1mm_ThermalVias, symbol Driver_Motor:DRV8871DDA
- added U2: INA226, Package_SO:VSSOP-10_3x3mm_P0.5mm, symbol Sensor_Energy:INA226
Connections:
- new net: U1.1 (GND), U1.7 (GND), U1.9 (GND)

Commit message: c
Parts:
- removed U1: DRV8871DDA, Package_SO:Texas_HTSOP-8-1EP_3.9x4.9mm_P1.27mm_EP2.95x4.9mm_Mask2.4x3.1mm_ThermalVias, symbol Driver_Motor:DRV8871DDA
Changed lines of the file:
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@@
-	)
-	(symbol
-		(lib_id "Driver_Motor:DRV8871DDA")
-		(at 204.47 90.17 0)
-		(unit 1)
-		(exclude_from_sim no)
-		(in_bom yes)
-		(on_board yes)
-		(dnp no)
-		(fields_autoplaced yes)
-		(property "Reference" "U1"
-			(at 206.6133 80.01 0)
-			(effects
-				(font
-					(size 1.27 1.27)
-				)
-				(justify left)
-			)
-		)
-		(property "Value" "DRV8871DDA"
-			(at 206.6133 82.55 0)
-			(effects
-				(font
-					(size 1.27 1.27)
-				)
-				(justify left)
-			)
-		)
-		(property "Footprint" "Package_SO:Texas_HTSOP-8-1EP_3.9x4.9mm_P1.27mm_EP2.95x4.9mm_Mask2.4x3.1mm_ThermalVias"
-			(at 210.82 91.44 0)
-			(effects
-				(font
-					(size 1.27 1.27)
-				)
-				(hide yes)
-			)
-		)
-		(property "Datasheet" "http://www.ti.com/lit/ds/symlink/drv8871.pdf"
-			(at 210.82 91.44 0)
-			(effects
-				(font
-					(size 1.27 1.27)
-				)
-				(hide yes)
-			)
-		)
-		(property "Description" "Brushed DC Motor Driver, PWM Control, 45V, 3.6A, Current limiting, HTSOP-8"
-			(at 204.47 90.17 0)
-			(effects
-				(font
-					(size 1.27 1.27)
-				)
-				(hide yes)
-			)
-		)
-		(pin "9"
-		)
-		(pin "6"
-		)
-		(pin "4"
-		)
-		(pin "3"
-		)
-		(pin "8"
-		)
-		(pin "1"
-		)
-		(pin "7"
-		)
-		(pin "2"
-		)
-		(pin "5"
-		)
-		(instances
-			(project ""
-				(path "/3fbae0b3-3e6a-4fc3-bce7-3e63a917950e"
-					(reference "U1")
-					(unit 1)
-				)
-			)
-		)
 	)
 	(symbol

Commit message: a
Parts:
- removed A1: Arduino_Nano_ESP32, Module:Arduino_Nano, symbol MCU_Module:Arduino_Nano_ESP32
- removed U2: INA226, Package_SO:VSSOP-10_3x3mm_P0.5mm, symbol Sensor_Energy:INA226
- added A2: Arduino_Nano_ESP32, Module:Arduino_Nano, symbol MCU_Module:Arduino_Nano_ESP32
- added D1: LED Auto, LED_THT:LED_D3.0mm, symbol Device:LED
- added D2: BAT3, LED_THT:LED_D3.0mm, symbol Device:LED
- added D3: BAT2, LED_THT:LED_D3.0mm, symbol Device:LED
- added D4: BAT1, LED_THT:LED_D3.0mm, symbol Device:LED
- added D5: MAN 3, LED_THT:LED_D3.0mm, symbol Device:LED
- added D6: MAN 2, LED_THT:LED_D3.0mm, symbol Device:LED
- added D7: MAN 1, LED_THT:LED_D3.0mm, symbol Device:LED
- added J4: Conn_01x02_Pin, symbol Connector:Conn_01x02_Pin
- added J4: VUSB/5V, Connector_PinHeader_2.54mm:PinHeader_1x01_P2.54mm_Horizontal, symbol Connector:Conn_01x01_Pin
- added J5: RESET, Connector_PinHeader_2.54mm:PinHeader_1x01_P2.54mm_Horizontal, symbol Connector:Conn_01x01_Pin
- added J5: Vin, Connector_PinHeader_2.54mm:PinHeader_1x01_P2.54mm_Horizontal, symbol Connector:Conn_01x01_Pin
- added J6: Motor Driver Pins, symbol Connector:Conn_01x04_Pin
- added R1, R2, R3, R4, R5, R6, R7: R, Resistor_THT:R_Axial_DIN0207_L6.3mm_D2.5mm_P7.62mm_Horizontal, symbol Device:R
- added SW1: Man+, Button_Switch_THT:SW_PUSH_6mm, symbol Switch:SW_Push
- added SW2: Man-, Button_Switch_THT:SW_PUSH_6mm, symbol Switch:SW_Push
- added SW3: Auto ON/OFF, Button_Switch_THT:SW_PUSH_6mm, symbol Switch:SW_Push
- added U1: INA226, Package_SO:VSSOP-10_3x3mm_P0.5mm, symbol Sensor_Energy:INA226
Connections:
- new net: A2.29 (GND), A2.4 (GND), D1.1 (K), D2.1 (K), D3.1 (K), D4.1 (K), D5.1 (K), D6.1 (K), D7.1 (K), SW1.1, SW2.2, SW3.2
- new net: D2.2 (A), R2.2
- new net: A2.26 (A7), SW1.2
- new net: D7.2 (A), R7.2
- new net: D6.2 (A), R6.2
- new net: A2.22 (A3), J6.1 (Pin_1)
- new net: A2.21 (A2), J6.2 (Pin_2)
- new net: A2.20 (A1), J6.3 (Pin_3)
- new net: A2.19 (A0), J6.4 (Pin_4)
- new net: D3.2 (A), R3.2
- new net: A2.12 (D9), R2.1
- new net: A2.9 (D6), R5.1
- new net: D5.2 (A), R5.2
- new net: A2.3 (~{RESET}), J5.1 (Pin_1)
- new net: A2.8 (D5), R6.1
- new net: A2.7 (D4), R7.1
- new net: A2.25 (A6), SW2.1
- new net: A2.27 (VUSB/5V), J4.1 (Pin_1)
- new net: A2.13 (D10/CS), R1.1
- new net: D1.2 (A), R1.2
- new net: A2.24 (SCL/A5), SW3.1
- new net: A2.30 (VIN), J5.1 (Pin_1)
- new net: D4.2 (A), R4.2
- new net: A2.10 (D7), R4.1
- new net: A2.11 (D8), R3.1
- new net i2c tmp: A2.5 (D2), A2.6 (D3), J4.1 (Pin_1), J4.2 (Pin_2)
- no-connect marks 0 -> 8

Commit message: main
Parts:
- removed J4: Conn_01x02_Pin, symbol Connector:Conn_01x02_Pin
- removed J4: VUSB/5V, Connector_PinHeader_2.54mm:PinHeader_1x01_P2.54mm_Horizontal, symbol Connector:Conn_01x01_Pin
- removed J5: RESET, Connector_PinHeader_2.54mm:PinHeader_1x01_P2.54mm_Horizontal, symbol Connector:Conn_01x01_Pin
- removed J5: Vin, Connector_PinHeader_2.54mm:PinHeader_1x01_P2.54mm_Horizontal, symbol Connector:Conn_01x01_Pin
- removed J6: Motor Driver Pins, symbol Connector:Conn_01x04_Pin
- removed SW1: Man+, Button_Switch_THT:SW_PUSH_6mm, symbol Switch:SW_Push
- removed SW2: Man-, Button_Switch_THT:SW_PUSH_6mm, symbol Switch:SW_Push
- removed SW3: Auto ON/OFF, Button_Switch_THT:SW_PUSH_6mm, symbol Switch:SW_Push
- added C1, C2: 10uF, Capacitor_SMD:C_1206_3216Metric, symbol Device:C
- added D8: US1M, Diode_SMD:D_SMA, symbol Diode:US1M
- added J4: Conn_01x04_Socket, Connector_PinHeader_2.54mm:PinHeader_1x04_P2.54mm_Vertical, symbol Connector:Conn_01x04_Socket
- added J7: Screw_Terminal_01x02, TerminalBlock_4Ucon:TerminalBlock_4Ucon_1x02_P3.50mm_Horizontal, symbol Connector:Screw_Terminal_01x02
- added R8, R9: R, Resistor_THT:R_Axial_DIN0207_L6.3mm_D2.5mm_P7.62mm_Horizontal, symbol Device:R
- added S1, S2, S3: SG06280N, SG06280N:SW_SG06280N, symbol SG06280N:SG06280N
Connections:
- net GND: now reaches A2.29 (GND), A2.4 (GND), D1.1 (K), D2.1 (K), D3.1 (K), D4.1 (K), D5.1 (K), D6.1 (K), D7.1 (K)
- net GND: now also J1.4, J2.4, J3.4, U1.7 (GND), C1.1, C2.1, J4.4 (Pin_4), J7.1 (Pin_1), S1.1, S2.1, S3.1
- net IN2: now reaches A2.26 (A7)
- net IN2: now also J4.2 (Pin_2)
- net SCL: now reaches J3.1
- net SCL: now also A2.24 (SCL/A5), J1.1, J2.1, U1.5 (SCL), R9.1
- net SDA: now reaches J3.2
- net SDA: now also A2.23 (SDA/A4), J1.2, J2.2, U1.4 (SDA), R8.1
- net +3.3V: now reaches J3.3
- net +3.3V: now also A2.17 (3V3), J1.3, J2.3, C1.2, R8.2, R9.2
- net IN1: now reaches A2.25 (A6)
- net IN1: now also J4.1 (Pin_1)
- net at R1.1: now also A2.6 (D3); no longer A2.13 (D10/CS)
- net at A2.30 (VIN): now also C2.2, D8.1 (K)
- net at A2.1 (D1/TX): now also S2.2
- net at A2.2 (D0/RX): now also S3.2
- net i2c tmp: no longer names the net of A2.5 (D2)
- net i2c tmp: now also S1.2; no longer A2.6 (D3)
- new net: D8.2 (A), J7.2 (Pin_2)
- no-connect marks 8 -> 5
Other:
- moved on the sheet: A2, D1, D2, D3, D4, D5, D6, D7, R1, R2, R3, R4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

Commit message: 2/9
Connections:
- net GND: now also S2.2, S3.2; no longer S2.1, S3.1
- net at A2.1 (D1/TX): no longer S2.2
- net at A2.2 (D0/RX): no longer S3.2
- net at A2.21 (A2): now also S3.1
- net at A2.22 (A3): now also S2.1
Other:
- moved on the sheet: S2, S3
Changed lines of the file:
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@@
 	(paper "User" 298.45 217.322)
-	(junction
-		(at 80.01 135.89)
-		(diameter 0)
-		(color 0 0 0 0)
-	)
 	(junction
 		(at 157.48 135.89)
@@
 	)
 	(junction
-		(at 59.69 135.89)
-		(diameter 0)
-		(color 0 0 0 0)
-	)
-	(junction
 		(at 120.65 135.89)
 		(diameter 0)
@@
 		(color 0 0 0 0)
 	)
+	(junction
+		(at 229.87 135.89)
+		(diameter 0)
+		(color 0 0 0 0)
+	)
 	(no_connect
 		(at 214.63 88.9)
@@
 	(wire
 		(pts
-			(xy 96.52 86.36) (xy 74.93 86.36)
-		)
-		(stroke
-			(width 0)
-			(type default)
-		)
-	)
-	(wire
-		(pts
-			(xy 36.83 81.28) (xy 36.83 135.89)
-		)
-		(stroke
-			(width 0)
-			(type default)
-		)
-	)
-	(wire
-		(pts
-			(xy 59.69 86.36) (xy 59.69 135.89)
-		)
-		(stroke
-			(width 0)
-			(type default)
-		)
-	)
-	(wire
-		(pts
-			(xy 179.07 88.9) (xy 96.52 88.9)
-		)
-		(stroke
-			(width 0)
-			(type default)
-		)
-	)
-	(wire
-		(pts
 			(xy 179.07 93.98) (xy 97.79 93.98)
 		)
@@
 	(wire
 		(pts
+			(xy 246.38 106.68) (xy 246.38 135.89)
+		)
+		(stroke
+			(width 0)
+			(type default)
+		)
+	)
+	(wire
+		(pts
 			(xy 97.79 135.89) (xy 110.49 135.89)
 		)
@@
 	(wire
 		(pts
+			(xy 246.38 135.89) (xy 229.87 135.89)
+		)
+		(stroke
+			(width 0)
+			(type default)
+		)
+	)
+	(wire
+		(pts
 			(xy 97.79 93.98) (xy 97.79 115.57)
 		)
@@
 	(wire
 		(pts
-			(xy 52.07 81.28) (xy 100.33 81.28)
+			(xy 229.87 109.22) (xy 229.87 135.89)
 		)
 		(stroke
@@
 	(wire
 		(pts
-			(xy 59.69 135.89) (xy 80.01 135.89)
-		)
-		(stroke
-			(width 0)
-			(type default)
-		)
-	)
-	(wire
-		(pts
 			(xy 80.01 135.89) (xy 97.79 135.89)
 		)
@@
 	(wire
 		(pts
+			(xy 229.87 135.89) (xy 196.85 135.89)
+		)
+		(stroke
+			(width 0)
+			(type default)
+		)
+	)
+	(wire
+		(pts
 			(xy 80.01 91.44) (xy 80.01 135.89)
 		)
@@
 	(wire
 		(pts
-			(xy 100.33 86.36) (xy 179.07 86.36)
-		)
-		(stroke
-			(width 0)
-			(type default)
-		)
-	)
-	(wire
-		(pts
 			(xy 139.7 104.14) (xy 139.7 115.57)
 		)
@@
 	(wire
 		(pts
-			(xy 96.52 88.9) (xy 96.52 86.36)
-		)
-		(stroke
-			(width 0)
-			(type default)
-		)
-	)
-	(wire
-		(pts
 			(xy 223.52 81.28) (xy 214.63 81.28)
 		)
@@
 	(wire
 		(pts
-			(xy 36.83 135.89) (xy 59.69 135.89)
+			(xy 214.63 106.68) (xy 231.14 106.68)
 		)
 		(stroke
@@
 		(pts
 			(xy 179.07 106.68) (xy 148.59 106.68)
-		)
-		(stroke
-			(width 0)
-			(type default)
-		)
-	)
-	(wire
-		(pts
-			(xy 100.33 81.28) (xy 100.33 86.36)
 		)
 		(stroke
@@
 	(symbol
 		(lib_id "SG06280N:SG06280N")
-		(at 67.31 86.36 0)
+		(at 222.25 109.22 0)
 		(unit 1)
 		(exclude_from_sim no)
@@
 		(fields_autoplaced yes)
 		(property "Reference" "S2"
-			(at 67.31 77.47 0)
+			(at 222.25 100.33 0)
 			(effects
 				(font
@@
 		)
 		(property "Value" "SG06280N"
-			(at 67.31 80.01 0)
+			(at 222.25 102.87 0)
 			(effects
 				(font
@@
 		)
 		(property "Footprint" "SG06280N:SW_SG06280N"
-			(at 67.31 86.36 0)
+			(at 222.25 109.22 0)
 			(effects
 				(font
@@
 		)
 		(property "Datasheet" ""
-			(at 67.31 86.36 0)
+			(at 222.25 109.22 0)
 			(effects
 				(font
@@
 		)
 		(property "Description" ""
-			(at 67.31 86.36 0)
+			(at 222.25 109.22 0)
 			(effects
 				(font
@@
 		)
 		(property "MF" "Snaptron"
-			(at 67.31 86.36 0)
+			(at 222.25 109.22 0)
 			(effects
 				(font
@@
 		)
 		(property "MAXIMUM_PACKAGE_HEIGHT" "0.33mm"
-			(at 67.31 86.36 0)
+			(at 222.25 109.22 0)
 			(effects
 				(font
@@
 		)
 		(property "CREATOR" "DIZAR"
-			(at 67.31 86.36 0)
+			(at 222.25 109.22 0)
 			(effects
 				(font
@@
 		)
 		(property "Price" "None"
-			(at 67.31 86.36 0)
+			(at 222.25 109.22 0)
 			(effects
 				(font
@@
 		)
 		(property "Package" "Package"
-			(at 67.31 86.36 0)
+			(at 222.25 109.22 0)
 			(effects
 				(font
@@
 		)
 		(property "Check_prices" "https://www.snapeda.com/parts/SG06280N/Snaptron/view-part/?ref=eda"
-			(at 67.31 86.36 0)
+			(at 222.25 109.22 0)
 			(effects
 				(font
@@
 		)
 		(property "STANDARD" "Manufacturer Recommendations"
-			(at 67.31 86.36 0)
+			(at 222.25 109.22 0)
 			(effects
 				(font
@@
 		)
 		(property "VERIFIER" ""
-			(at 67.31 86.36 0)
+			(at 222.25 109.22 0)
 			(effects
 				(font
@@
 		)
 		(property "SnapEDA_Link" "https://www.snapeda.com/parts/SG06280N/Snaptron/view-part/?ref=snap"
-			(at 67.31 86.36 0)
+			(at 222.25 109.22 0)
 			(effects
 				(font
@@
 		)
 		(property "MP" "SG06280N"
-			(at 67.31 86.36 0)
+			(at 222.25 109.22 0)
 			(effects
 				(font
@@
 		)
 		(property "Description_1" "SMT TACTILE DOME SWITCH SPST-NO"
-			(at 67.31 86.36 0)
+			(at 222.25 109.22 0)
 			(effects
 				(font
@@
 		)
 		(property "Availability" "Not in stock"
-			(at 67.31 86.36 0)
+			(at 222.25 109.22 0)
 			(effects
 				(font
@@
 		)
 		(property "MANUFACTURER" "Snaptron"
-			(at 67.31 86.36 0)
+			(at 222.25 109.22 0)
 			(effects
 				(font
@@
 	(symbol
 		(lib_id "SG06280N:SG06280N")
-		(at 44.45 81.28 0)
+		(at 238.76 106.68 0)
 		(unit 1)
 		(exclude_from_sim no)
@@
 		(fields_autoplaced yes)
 		(property "Reference" "S3"
-			(at 44.45 72.39 0)
+			(at 238.76 97.79 0)
 			(effects
 				(font
@@
 		)
 		(property "Value" "SG06280N"
-			(at 44.45 74.93 0)
+			(at 238.76 100.33 0)
 			(effects
 				(font
@@
 		)
 		(property "Footprint" "SG06280N:SW_SG06280N"
-			(at 44.45 81.28 0)
+			(at 238.76 106.68 0)
 			(effects
 				(font
@@
 		)
 		(property "Datasheet" ""
-			(at 44.45 81.28 0)
+			(at 238.76 106.68 0)
 			(effects
 				(font
@@
 		)
 		(property "Description" ""
-			(at 44.45 81.28 0)
+			(at 238.76 106.68 0)
 			(effects
 				(font
@@
 		)
 		(property "MF" "Snaptron"
-			(at 44.45 81.28 0)
+			(at 238.76 106.68 0)
 			(effects
 				(font
@@
 		)
 		(property "MAXIMUM_PACKAGE_HEIGHT" "0.33mm"
-			(at 44.45 81.28 0)
+			(at 238.76 106.68 0)
 			(effects
 				(font
@@
 		)
 		(property "CREATOR" "DIZAR"
-			(at 44.45 81.28 0)
+			(at 238.76 106.68 0)
 			(effects
 				(font
@@
 		)
 		(property "Price" "None"
-			(at 44.45 81.28 0)
+			(at 238.76 106.68 0)
 			(effects
 				(font
@@
 		)
 		(property "Package" "Package"
-			(at 44.45 81.28 0)
+			(at 238.76 106.68 0)
 			(effects
 				(font
@@
 		)
 		(property "Check_prices" "https://www.snapeda.com/parts/SG06280N/Snaptron/view-part/?ref=eda"
-			(at 44.45 81.28 0)
+			(at 238.76 106.68 0)
 			(effects
 				(font
@@
 		)
 		(property "STANDARD" "Manufacturer Recommendations"
-			(at 44.45 81.28 0)
+			(at 238.76 106.68 0)
 			(effects
 				(font
@@
 		)
 		(property "VERIFIER" ""
-			(at 44.45 81.28 0)
+			(at 238.76 106.68 0)
 			(effects
 				(font
@@
 		)
 		(property "SnapEDA_Link" "https://www.snapeda.com/parts/SG06280N/Snaptron/view-part/?ref=snap"
-			(at 44.45 81.28 0)
+			(at 238.76 106.68 0)
 			(effects
 				(font
@@
 		)
 		(property "MP" "SG06280N"
-			(at 44.45 81.28 0)
+			(at 238.76 106.68 0)
 			(effects
 				(font
@@
 		)
 		(property "Description_1" "SMT TACTILE DOME SWITCH SPST-NO"
-			(at 44.45 81.28 0)
+			(at 238.76 106.68 0)
 			(effects
 				(font
@@
 		)
 		(property "Availability" "Not in stock"
-			(at 44.45 81.28 0)
+			(at 238.76 106.68 0)
 			(effects
 				(font
@@
 		)
 		(property "MANUFACTURER" "Snaptron"
-			(at 44.45 81.28 0)
-			(effects
-				(font
+			(at 238.76 106.68 0)
+			(effects
+				(font

Commit message: 2/9/26
Parts:
- added C3: 0.1uF, Capacitor_SMD:C_1206_3216Metric, symbol Device:C
Connections:
- net +3.3V: now also U1.6 (VS), C3.2
- net GND: now also C3.1
- no-connect marks 5 -> 7
Other:
- moved on the sheet: A2, C1, C2, D1, D2, D3, D4, D5, D6, D7, D8, J7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

Commit message: a
Parts:
- removed S1, S2, S3: SG06280N, SG06280N:SW_SG06280N, symbol SG06280N:SG06280N
- added S1, S2, S3: TL3315NF250Q, TL3315NF250Q:SW_TL3315NF250Q, symbol TL3315NF250Q:TL3315NF250Q
Connections:
- net GND: now also S1.3, S1.4, S2.3, S2.4, S3.1, S3.2
- net at A2.22 (A3): now also S2.1, S2.2
- net at A2.21 (A2): now also S1.1, S1.2
- net at A2.5 (D2): now also S3.3, S3.4

Commit message: 2/13
Parts:
- removed FID3, FID4: FIDUCIAL_1MM, coolerpcb:FIDUCIAL_1MM, symbol coolerpcb-eagle-import:FIDUCIAL_1MM
- removed J1, J2, J3: S4B-PH-SM4-TB, S4B-PH-SM4-TB:JST_S4B-PH-SM4-TB, symbol S4B-PH-SM4-TB:S4B-PH-SM4-TB
- removed U$1, U$17, U$19, U$21: MOUNTINGHOLE2.5, coolerpcb:MOUNTINGHOLE_2.5_PLATED, symbol coolerpcb-eagle-import:MOUNTINGHOLE2.5
- added J1, J2, J5: SS-12800-009, SS_12800_009:STEWART_SS-12800-009, symbol SS-12800-009:SS-12800-009
- added J3: Screw_Terminal_01x02, TerminalBlock_4Ucon:TerminalBlock_4Ucon_1x02_P3.50mm_Horizontal, symbol Connector:Screw_Terminal_01x02
- added JP1, JP2, JP3, JP4, JP5, JP6: SolderJumper_2_Open, Jumper:SolderJumper-2_P1.3mm_Open_TrianglePad1.0x1.5mm, symbol Jumper:SolderJumper_2_Open
- added R10: 68m, Resistor_SMD:R_1206_3216Metric, symbol Device:R
- added R11: 100m, Resistor_SMD:R_1206_3216Metric, symbol Device:R
- added R12: 120m, Resistor_SMD:R_1206_3216Metric, symbol Device:R
- added U2: DRV8871DDA, Package_SO:Texas_HTSOP-8-1EP_3.9x4.9mm_P1.27mm_EP2.95x4.9mm_Mask2.4x3.1mm_ThermalVias, symbol Driver_Motor:DRV8871DDA
- added U4: XTPS55285VALR, footprints:VAL0015A-MFG, symbol 2026-02-14_03-24-54:XTPS55285VALR
- D1, D2, D3, D4, D5, D6, D7: footprint LED_THT:LED_D3.0mm -> LED_SMD:LED_1206_3216Metric
- R1, R2, R3, R4, R5, R6, R7: value R -> 220; footprint Resistor_THT:R_Axial_DIN0207_L6.3mm_D2.5mm_P7.62mm_Horizontal -> Resistor_SMD:R_1206_3216Metric
- R8, R9: footprint Resistor_THT:R_Axial_DIN0207_L6.3mm_D2.5mm_P7.62mm_Horizontal -> Resistor_SMD:R_1206_3216Metric
Connections:
- net +3.3V: now also J1.2, J2.2, J5.2
- net GND: now also U1.1 (A1), U1.2 (A0), J1.1, J1.SH1 (SHIELD), J1.SH2 (SHIELD__1), J2.1, J2.SH1 (SHIELD), J2.SH2 (SHIELD__1), J5.1, J5.SH1 (SHIELD), J5.SH2 (SHIELD__1)
- net SCL: now also J1.4, J2.4, J5.4
- net SDA: now also J1.3, J2.3, J5.3
- net at U1.10 (Vin+): now also JP2.2 (B), JP4.2 (B), JP6.2 (B)
- net at U1.8 (Vbus): now also U1.9 (Vin-), JP1.1 (A), JP3.1 (A), JP5.1 (A)
- new net: JP1.2 (B), R10.2
- new net: JP2.1 (A), R10.1
- new net: JP6.1 (A), R12.1
- new net: JP5.2 (B), R12.2
- new net: JP4.1 (A), R11.1
- new net: JP3.2 (B), R11.2
- new net: U2.1 (GND), U2.7 (GND), U2.9 (GND)
- no-connect marks 7 -> 6
Other:
- moved on the sheet: A2, C1, C2, D1, D2, D3, D4, D5, D6, D7, D8, J7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
