File: MainPCB/MAIN_PCB.kicad_sch (KiCad schematic)
At the start: 34 parts, among them U1 INA226, U2 DRV8871DDA

Commit message: n
Connections:
- net +BATT: no longer J-Battery1.1, R10.1, U1.10 (Vin+)
- net GND: now also J-Battery1.3
- net GNDPWR: no longer J-Battery1.3
- new net: J-Battery1.1, R10.1, U1.10 (Vin+)
- no-connect marks 10 -> 9
Changed lines of the file:
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@@
 	)
 	(junction
-		(at 46.99 49.53)
-		(diameter 0)
-		(color 0 0 0 0)
-	)
-	(junction
 		(at 251.46 53.34)
 		(diameter 0)
@@
 	)
 	(junction
-		(at 64.77 58.42)
-		(diameter 0)
-		(color 0 0 0 0)
-	)
-	(junction
 		(at 73.66 165.1)
 		(diameter 0)
@@
 	)
 	(no_connect
-		(at 190.5 113.03)
-	)
-	(no_connect
 		(at 190.5 146.05)
 	)
@@
 	(wire
 		(pts
-			(xy 64.77 58.42) (xy 57.15 58.42)
-		)
-		(stroke
-			(width 0)
-			(type default)
-		)
-	)
-	(wire
-		(pts
 			(xy 86.36 48.26) (xy 86.36 50.8)
 		)
@@
 	(wire
 		(pts
-			(xy 64.77 58.42) (xy 64.77 60.96)
+			(xy 46.99 49.53) (xy 57.15 49.53)
 		)
 		(stroke
@@
 	(wire
 		(pts
-			(xy 55.88 165.1) (xy 73.66 165.1)
+			(xy 64.77 46.99) (xy 64.77 60.96)
 		)
 		(stroke
@@
 	(wire
 		(pts
-			(xy 96.52 128.27) (xy 154.94 128.27)
+			(xy 55.88 165.1) (xy 73.66 165.1)
 		)
 		(stroke
@@
 	(wire
 		(pts
-			(xy 172.72 156.21) (xy 172.72 165.1)
+			(xy 96.52 128.27) (xy 154.94 128.27)
 		)
 		(stroke
@@
 	(wire
 		(pts
-			(xy 106.68 160.02) (xy 106.68 165.1)
+			(xy 172.72 156.21) (xy 172.72 165.1)
 		)
 		(stroke
@@
 	(wire
 		(pts
-			(xy 46.99 49.53) (xy 64.77 49.53)
+			(xy 106.68 160.02) (xy 106.68 165.1)
 		)
 		(stroke
@@
 	(wire
 		(pts
-			(xy 201.93 143.51) (xy 190.5 143.51)
+			(xy 46.99 46.99) (xy 64.77 46.99)
 		)
 		(stroke
@@
 	(wire
 		(pts
-			(xy 86.36 125.73) (xy 154.94 125.73)
+			(xy 201.93 143.51) (xy 190.5 143.51)
 		)
 		(stroke
@@
 	(wire
 		(pts
-			(xy 213.36 138.43) (xy 190.5 138.43)
+			(xy 86.36 125.73) (xy 154.94 125.73)
 		)
 		(stroke
@@
 	(wire
 		(pts
-			(xy 251.46 53.34) (xy 251.46 50.8)
+			(xy 213.36 138.43) (xy 190.5 138.43)
 		)
 		(stroke
@@
 	(wire
 		(pts
-			(xy 64.77 49.53) (xy 64.77 58.42)
+			(xy 251.46 53.34) (xy 251.46 50.8)
 		)
 		(stroke
@@
 	(wire
 		(pts
-			(xy 57.15 58.42) (xy 57.15 69.85)
-		)
-		(stroke
-			(width 0)
-			(type default)
-		)
-	)
-	(wire
-		(pts
-			(xy 46.99 46.99) (xy 46.99 49.53)
+			(xy 57.15 49.53) (xy 57.15 69.85)
 		)
 		(stroke
@@
 		)
 	)
-	(wire
-		(pts
-			(xy 46.99 52.07) (xy 46.99 54.61)
-		)
-		(stroke
-			(width 0)
-			(type default)
-		)
-	)
 	(global_label "SCL"
 		(shape input)
@@
 					(unit 1)
 				)
+			)
+		)
+	)
+	(symbol
+		(lib_id "power:GND")
+		(at 46.99 52.07 90)
+		(unit 1)
+		(exclude_from_sim no)
+		(in_bom yes)
+		(on_board yes)
+		(dnp no)
+		(fields_autoplaced yes)
+		(property "Reference" "#PWR015"
+			(at 53.34 52.07 0)
+			(effects
+				(font
+					(size 1.27 1.27)
+				)
+				(hide yes)
+			)
+		)
+		(property "Value" "GND"
+			(at 50.8 52.0699 90)
+			(effects
+				(font
+					(size 1.27 1.27)
+				)
+				(justify right)
+			)
+		)
+		(property "Footprint" ""
+			(at 46.99 52.07 0)
+			(effects
+				(font
+					(size 1.27 1.27)
+				)
+				(hide yes)
+			)
+		)
+		(property "Datasheet" ""
+			(at 46.99 52.07 0)
+			(effects
+				(font
+					(size 1.27 1.27)
+				)
+				(hide yes)
+			)
+		)
+		(property "Description" "Power symbol creates a global label with name \"GND\" , ground"
+			(at 46.99 52.07 0)
+			(effects
+				(font
+					(size 1.27 1.27)
+				)
+				(hide yes)
+			)
+		)
+		(pin "1"
+		)
+		(instances
+			(project "MAIN_PCB"
+				(path "/3fbae0b3-3e6a-4fc3-bce7-3e63a917950e"
+					(reference "#PWR015")
+					(unit 1)
+				)

Commit message: Nate
Parts:
- removed A2: Arduino_Nano_ESP32, Module:Arduino_Nano, symbol MCU_Module:Arduino_Nano_ESP32
- added A1: Arduino_Nano_ESP32, Module:Arduino_Nano, symbol MCU_Module:Arduino_Nano_ESP32
- added C5, C6: C, symbol Device:C
- R1, R2, R3, R4, R5, R6, R7: value 220 -> R; footprint Resistor_SMD:R_1206_3216Metric -> (none)
Connections:
- net +3.3V: now also A1.17 (3V3)
- net GND: now also A1.29 (GND), A1.4 (GND), C5.1, C6.1
- net PWM: now also A1.20 (A1)
- net SCL: now also A1.24 (SCL/A5)
- net SDA: now also A1.23 (SDA/A4)
- net Vdrive: now also C5.2, C6.2
- net at D2.2 (A): now also R7.2; no longer R2.2
- net at D7.2 (A): now also R2.2; no longer R7.2
- net at D6.2 (A): now also R3.2; no longer R6.2
- net at D3.2 (A): now also R6.2; no longer R3.2
- net at C2.1, L2.2: now also A1.30 (VIN)
- net at R2.1: now also A1.7 (D4)
- net at R5.1: now also A1.10 (D7)
- net at R5.2: now also D4.2 (A); no longer D5.2 (A)
- net at R6.1: now also A1.11 (D8)
- net at R7.1: now also A1.12 (D9)
- net at S2.1, S2.2: now also A1.22 (A3)
- net at R1.1: now also A1.6 (D3)
- net at S3.3, S3.4: now also A1.5 (D2)
- net at S1.1, S1.2: now also A1.21 (A2)
- net at R4.2: now also D5.2 (A); no longer D4.2 (A)
- net at R4.1: now also A1.9 (D6)
- net at R3.1: now also A1.8 (D5)

Commit message: Nate
Parts:
- removed D8, D9: US1M, Diode_SMD:D_SMA, symbol Diode:US1M
- added C7: 10u, symbol Device:C
- added CR1: SA15CA, DO-204AC_SA, symbol 2026-03-08_02-43-44:SA15CA
- added D8, D9: 80SQ045NRLG, DIOAD2860W130L840D505, symbol 80SQ045NRLG:80SQ045NRLG
- C1, C3: footprint Capacitor_SMD:C_1206_3216Metric -> (none)
- C5: value C -> 0.1u
- C6: value C -> 100u
- R1, R2, R3, R4, R5, R6, R7: value R -> 56; footprint (none) -> Resistor_THT:R_Axial_DIN0207_L6.3mm_D2.5mm_P7.62mm_Horizontal
- R13, R8, R9: footprint Resistor_SMD:R_1206_3216Metric -> Resistor_THT:R_Axial_DIN0207_L6.3mm_D2.5mm_P7.62mm_Horizontal
Connections:
- net +BATT: now also D8.2 (A)
- net DRV: now also CR1.2
- net GND: now also C7.1
- net GNDPWR: now also D9.2 (A)
- net RTN: now also CR1.1
- net Vdrive: now also C7.2, D9.1 (K)
- net at C4.1, L2.1: now also D8.1 (K)
Other:
- moved on the sheet: C5, C6, J-Pump1, R13, U2

Commit message: 3/8
Parts:
- removed J-TMP1: 861-004-213R00Y, 861.preety:861-004-213R00Y, symbol SS-12800-009:SS-12800-009
- added J-TMP117: 861-004-213R00Y, 861.preety:861-004-213R00Y, symbol SS-12800-009:SS-12800-009
- C1, C6, C7: footprint (none) -> Capacitor_THT:CP_Radial_D5.0mm_P2.00mm
- C3, C5: footprint (none) -> CAP_BF01:CAP_BF01_AVX
- CR1: footprint DO-204AC_SA -> DO-204AC_SA:DO-204AC_SA
- D1, D2, D3, D4, D5, D6, D7: footprint LED_SMD:LED_1206_3216Metric -> LED_THT:LED_Oval_W5.2mm_H3.8mm
- D8, D9: footprint DIOAD2860W130L840D505 -> 80SQ045NRLG:DIOAD2860W130L840D505
- J-Battery1, J-Pump1: MANUFACTURER Stewart Connector -> NorComp Connector; MAXIMUM_PACKAGE_HEIGHT 12.7mm -> 10.5mm
- L2: footprint IND_LQH44PN:IND_LQH44PN_PR_MUR-L -> IND_LQH44PN:IND_LQH44PN_PR_MUR
Connections:
- net +3.3V: now also J-TMP117.2
- net DRV: now also CR1.1; no longer CR1.2
- net GND: now also J-TMP117.1
- net GNDPWR: now also J-TMP117.SH1 (SHIELD), J-TMP117.SH2 (SHIELD__1)
- net RTN: now also CR1.2; no longer CR1.1
- net SCL: now also J-TMP117.4
- net SDA: now also J-TMP117.3
Other:
- moved on the sheet: CR1, J-Battery1

Commit message: Nate
Changed lines of the file:
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@@
-	(wire
-		(pts
-			(xy 140.97 59.69) (xy 139.7 59.69)
-		)
-		(stroke
-			(width 0)
-			(type default)
-		)
-	)
 	(wire
 		(pts
@@
 	(wire
 		(pts
-			(xy 140.97 69.85) (xy 149.86 69.85)
-		)
-		(stroke
-			(width 0)
-			(type default)
-		)
-	)
-	(wire
-		(pts
 			(xy 238.76 165.1) (xy 228.6 165.1)
 		)
@@
 		(pts
 			(xy 213.36 138.43) (xy 190.5 138.43)
-		)
-		(stroke
-			(width 0)
-			(type default)
-		)
-	)
-	(wire
-		(pts
-			(xy 140.97 69.85) (xy 140.97 59.69)
 		)
 		(stroke
@@
 					(unit 1)
 				)
+			)
+		)
+	)
+	(symbol
+		(lib_id "power:GND")
+		(at 139.7 59.69 270)
+		(unit 1)
+		(exclude_from_sim no)
+		(in_bom yes)
+		(on_board yes)
+		(dnp no)
+		(fields_autoplaced yes)
+		(property "Reference" "#PWR022"
+			(at 133.35 59.69 0)
+			(effects
+				(font
+					(size 1.27 1.27)
+				)
+				(hide yes)
+			)
+		)
+		(property "Value" "GND"
+			(at 135.89 59.6899 90)
+			(effects
+				(font
+					(size 1.27 1.27)
+				)
+				(justify right)
+			)
+		)
+		(property "Footprint" ""
+			(at 139.7 59.69 0)
+			(effects
+				(font
+					(size 1.27 1.27)
+				)
+				(hide yes)
+			)
+		)
+		(property "Datasheet" ""
+			(at 139.7 59.69 0)
+			(effects
+				(font
+					(size 1.27 1.27)
+				)
+				(hide yes)
+			)
+		)
+		(property "Description" "Power symbol creates a global label with name \"GND\" , ground"
+			(at 139.7 59.69 0)
+			(effects
+				(font
+					(size 1.27 1.27)
+				)
+				(hide yes)
+			)
+		)
+		(pin "1"
+		)
+		(instances
+			(project "MAIN_PCB"
+				(path "/3fbae0b3-3e6a-4fc3-bce7-3e63a917950e"
+					(reference "#PWR022")
+					(unit 1)
+				)

Commit message: nate
Parts:
- added C8: 0.1uF, CAP_BF01:CAP_BF01_AVX, symbol Device:C
- added R11: Shunt, Resistor_SMD:R_1206_3216Metric, symbol Device:R
- added R12: 100k, Resistor_THT:R_Axial_DIN0207_L6.3mm_D2.5mm_P10.16mm_Horizontal, symbol Device:R
- added R14: 390k, Resistor_THT:R_Axial_DIN0207_L6.3mm_D2.5mm_P10.16mm_Horizontal, symbol Device:R
- added U3: INA226, Package_SO:VSSOP-10_3x3mm_P0.5mm, symbol Sensor_Energy:INA226
- R1, R13, R2, R3, R4, R5, R6, R7, R8, R9: footprint Resistor_THT:R_Axial_DIN0207_L6.3mm_D2.5mm_P7.62mm_Horizontal -> Resistor_THT:R_Axial_DIN0207_L6.3mm_D2.5mm_P10.16mm_Horizontal
- R10: value 100m -> Shunt
Connections:
- net +3.3V: now also C8.2, U3.2 (A0), U3.6 (VS)
- net +BATT: now also R11.2, R14.1, U3.8 (Vbus), U3.9 (Vin-); no longer J-Battery1.2
- net GND: now also C8.1, R12.2, U3.1 (A1), U3.7 (GND); no longer C5.1, C6.1, C7.1
- net GNDPWR: now also C5.1, C6.1, C7.1
- net PWM: now also A1.19 (A0); no longer A1.20 (A1)
- net SCL: now also U3.5 (SCL)
- net SDA: now also U3.4 (SDA)
- new net: A1.20 (A1), R12.1, R14.2
- new net: J-Battery1.2, R11.1, U3.10 (Vin+)
Other:
- note added: "Current Sensors"
- note removed: "Current Sense"
- moved on the sheet: A1, C1, C2, C4, D1, D2, D3, D4, D5, D6, D7, D8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

Commit message: DRV8871
Connections:
- net +3.3V: now also C1.1; no longer C1.2
- net GND: now also C1.2, C5.1, C7.2; no longer C1.1
- net GNDPWR: now also C6.2; no longer C5.1, C6.1, C7.1
- net Vdrive: now also C6.1, C7.1; no longer C6.2, C7.2
Other:
- moved on the sheet: C1, C6, C7
Changed lines of the file:
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@@
 	)
 	(junction
+		(at 134.62 52.07)
+		(diameter 0)
+		(color 0 0 0 0)
+	)
+	(junction
 		(at 265.43 165.1)
 		(diameter 0)
@@
 	)
 	(junction
+		(at 236.22 110.49)
+		(diameter 0)
+		(color 0 0 0 0)
+	)
+	(junction
 		(at 128.27 52.07)
 		(diameter 0)
@@
 	)
 	(junction
-		(at 140.97 52.07)
-		(diameter 0)
-		(color 0 0 0 0)
-	)
-	(junction
 		(at 245.11 123.19)
 		(diameter 0)
@@
 	)
 	(junction
-		(at 134.62 52.07)
-		(diameter 0)
-		(color 0 0 0 0)
-	)
-	(junction
 		(at 254 45.72)
 		(diameter 0)
@@
 	)
 	(junction
-		(at 252.73 140.97)
+		(at 140.97 52.07)
 		(diameter 0)
 		(color 0 0 0 0)
 	)
 	(junction
-		(at 139.7 62.23)
+		(at 252.73 140.97)
 		(diameter 0)
 		(color 0 0 0 0)
 	)
 	(junction
-		(at 251.46 59.69)
+		(at 139.7 62.23)
 		(diameter 0)
 		(color 0 0 0 0)
 	)
 	(junction
-		(at 236.22 110.49)
+		(at 251.46 59.69)
 		(diameter 0)
 		(color 0 0 0 0)
@@
 	(wire
 		(pts
+			(xy 134.62 52.07) (xy 140.97 52.07)
+		)
+		(stroke
+			(width 0)
+			(type default)
+		)
+	)
+	(wire
+		(pts
 			(xy 110.49 165.1) (xy 123.19 165.1)
 		)
@@
 	(wire
 		(pts
-			(xy 167.64 64.77) (xy 167.64 69.85)
+			(xy 236.22 110.49) (xy 241.3 110.49)
 		)
 		(stroke
@@
 	(wire
 		(pts
-			(xy 243.84 123.19) (xy 245.11 123.19)
+			(xy 167.64 64.77) (xy 167.64 69.85)
 		)
 		(stroke
@@
 	(wire
 		(pts
-			(xy 152.4 133.35) (xy 152.4 144.78)
+			(xy 243.84 123.19) (xy 245.11 123.19)
 		)
 		(stroke
@@
 	(wire
 		(pts
-			(xy 92.71 22.86) (xy 92.71 25.4)
+			(xy 152.4 133.35) (xy 152.4 144.78)
 		)
 		(stroke
@@
 	(wire
 		(pts
-			(xy 143.51 165.1) (xy 152.4 165.1)
+			(xy 92.71 22.86) (xy 92.71 25.4)
 		)
 		(stroke
@@
 	(wire
 		(pts
-			(xy 161.29 135.89) (xy 161.29 144.78)
+			(xy 143.51 165.1) (xy 152.4 165.1)
 		)
 		(stroke
@@
 	(wire
 		(pts
-			(xy 124.46 52.07) (xy 128.27 52.07)
+			(xy 161.29 135.89) (xy 161.29 144.78)
 		)
 		(stroke
@@
 	(wire
 		(pts
-			(xy 161.29 165.1) (xy 170.18 165.1)
+			(xy 124.46 52.07) (xy 128.27 52.07)
 		)
 		(stroke
@@
 	(wire
 		(pts
-			(xy 134.62 52.07) (xy 140.97 52.07)
+			(xy 161.29 165.1) (xy 170.18 165.1)
 		)
 		(stroke
@@
 	(wire
 		(pts
-			(xy 241.3 110.49) (xy 236.22 110.49)
-		)
-		(stroke
-			(width 0)
-			(type default)
-		)
-	)
-	(wire
-		(pts
 			(xy 49.53 33.02) (xy 71.12 33.02)
 		)
@@
 	(wire
 		(pts
-			(xy 236.22 110.49) (xy 227.33 110.49)
+			(xy 227.33 110.49) (xy 236.22 110.49)
 		)
 		(stroke
@@
 	(wire
 		(pts
-			(xy 250.19 138.43) (xy 227.33 138.43)
+			(xy 140.97 52.07) (xy 149.86 52.07)
 		)
 		(stroke
@@
 	(wire
 		(pts
-			(xy 133.35 165.1) (xy 143.51 165.1)
+			(xy 250.19 138.43) (xy 227.33 138.43)
 		)
 		(stroke
@@
 	(wire
 		(pts
-			(xy 227.33 135.89) (xy 260.35 135.89)
+			(xy 133.35 165.1) (xy 143.51 165.1)
 		)
 		(stroke
@@
 	(wire
 		(pts
-			(xy 81.28 33.02) (xy 82.55 33.02)
+			(xy 227.33 135.89) (xy 260.35 135.89)
 		)
 		(stroke
@@
 	(wire
 		(pts
-			(xy 254 54.61) (xy 254 57.15)
+			(xy 81.28 33.02) (xy 82.55 33.02)
 		)
 		(stroke
@@
 	(wire
 		(pts
-			(xy 123.19 165.1) (xy 133.35 165.1)
+			(xy 254 54.61) (xy 254 57.15)
 		)
 		(stroke
@@
 	(wire
 		(pts
-			(xy 140.97 52.07) (xy 149.86 52.07)
+			(xy 123.19 165.1) (xy 133.35 165.1)
 		)
 		(stroke
@@
 	)
 	(symbol
-		(lib_id "power:GNDPWR")
-		(at 128.27 44.45 180)
-		(unit 1)
-		(exclude_from_sim no)
-		(in_bom yes)
-		(on_board yes)
-		(dnp no)
-		(fields_autoplaced yes)
-		(property "Reference" "#PWR018"
-			(at 128.27 39.37 0)
-			(effects
-				(font
-					(size 1.27 1.27)
-				)
-				(hide yes)
-			)
-		)
-		(property "Value" "GNDPWR"
-			(at 128.397 40.64 0)
-			(effects
-				(font
-					(size 1.27 1.27)
-				)
-			)
-		)
-		(property "Footprint" ""
-			(at 128.27 43.18 0)
-			(effects
-				(font
-					(size 1.27 1.27)
-				)
-				(hide yes)
-			)
-		)
-		(property "Datasheet" ""
-			(at 128.27 43.18 0)
-			(effects
-				(font
-					(size 1.27 1.27)
-				)
-				(hide yes)
-			)
-		)
-		(property "Description" "Power symbol creates a global label with name \"GNDPWR\" , global ground"
-			(at 128.27 44.45 0)
-			(effects
-				(font
-					(size 1.27 1.27)
-				)
-				(hide yes)
-			)
-		)
-		(pin "1"
-		)
-		(instances
-			(project "MAIN_PCB"
-				(path "/3fbae0b3-3e6a-4fc3-bce7-3e63a917950e"
-					(reference "#PWR018")
-					(unit 1)
-				)
-			)
-		)
-	)
-	(symbol
 		(lib_id "TL3315NF250Q:TL3315NF250Q")
 		(at 257.81 138.43 0)
@@
 	(symbol
 		(lib_id "Device:C")
-		(at 140.97 48.26 0)
+		(at 140.97 48.26 180)
 		(unit 1)
 		(exclude_from_sim no)
@@
 					(size 1.27 1.27)
 				)
-				(justify left)
+				(justify right)
 			)
 		)
@@
 					(size 1.27 1.27)
 				)
-				(justify left)
+				(justify right)
 			)
 		)
 		(property "Footprint" "Capacitor_THT:CP_Radial_D5.0mm_P2.00mm"
-			(at 141.9352 52.07 0)
+			(at 140.0048 44.45 0)
 			(effects
 				(font
@@
 	)
 	(symbol
-		(lib_id "power:GNDPWR")
+		(lib_id "power:GND")
 		(at 134.62 44.45 180)
 		(unit 1)
@@
 		(fields_autoplaced yes)
 		(property "Reference" "#PWR019"
-			(at 134.62 39.37 0)
+			(at 134.62 38.1 0)
 			(effects
 				(font
@@
 			)
 		)
-		(property "Value" "GNDPWR"
-			(at 134.747 40.64 0)
+		(property "Value" "GND"
+			(at 134.62 39.37 0)
 			(effects
 				(font
@@
 		)
 		(property "Footprint" ""
-			(at 134.62 43.18 0)
+			(at 134.62 44.45 0)
 			(effects
 				(font
@@
 		)
 		(property "Datasheet" ""
-			(at 134.62 43.18 0)
+			(at 134.62 44.45 0)
 			(effects
 				(font
@@
 			)
 		)
-		(property "Description" "Power symbol creates a global label with name \"GNDPWR\" , global ground"
+		(property "Description" "Power symbol creates a global label with name \"GND\" , ground"
 			(at 134.62 44.45 0)
 			(effects
@@
 	)
 	(symbol
+		(lib_id "power:GND")
+		(at 128.27 44.45 180)
+		(unit 1)
+		(exclude_from_sim no)
+		(in_bom yes)
+		(on_board yes)
+		(dnp no)
+		(fields_autoplaced yes)
+		(property "Reference" "#PWR018"
+			(at 128.27 38.1 0)
+			(effects
+				(font
+					(size 1.27 1.27)
+				)
+				(hide yes)
+			)
+		)
+		(property "Value" "GND"
+			(at 128.27 39.37 0)
+			(effects
+				(font
+					(size 1.27 1.27)
+				)
+			)
+		)
+		(property "Footprint" ""
+			(at 128.27 44.45 0)
+			(effects
+				(font
+					(size 1.27 1.27)
+				)
+				(hide yes)
+			)
+		)
+		(property "Datasheet" ""
+			(at 128.27 44.45 0)
+			(effects
+				(font
+					(size 1.27 1.27)
+				)
+				(hide yes)
+			)
+		)
+		(property "Description" "Power symbol creates a global label with name \"GND\" , ground"
+			(at 128.27 44.45 0)
+			(effects
+				(font
+					(size 1.27 1.27)
+				)
+				(hide yes)
+			)
+		)
+		(pin "1"
+		)
+		(instances
+			(project "MAIN_PCB"
+				(path "/3fbae0b3-3e6a-4fc3-bce7-3e63a917950e"
+					(reference "#PWR018")
+					(unit 1)
+				)
+			)
+		)
+	)
+	(symbol
 		(lib_id "Device:C")
-		(at 134.62 48.26 0)
+		(at 134.62 48.26 180)
 		(unit 1)
 		(exclude_from_sim no)
@@
 					(size 1.27 1.27)
 				)
-				(justify left)
+				(justify right)
 			)
 		)
@@
 					(size 1.27 1.27)
 				)
-				(justify left)
+				(justify right)
 			)
 		)
 		(property "Footprint" "Capacitor_THT:CP_Radial_D5.0mm_P2.00mm"
-			(at 135.5852 52.07 0)
+			(at 133.6548 44.45 0)
 			(effects
 				(font
@@
 	(symbol
 		(lib_id "Device:C")
-		(at 236.22 106.68 0)
+		(at 236.22 106.68 180)
 		(unit 1)
 		(exclude_from_sim no)
@@
 					(size 1.27 1.27)
 				)
-				(justify left)
+				(justify right)
 			)
 		)
@@
 					(size 1.27 1.27)
 				)
-				(justify left)
+				(justify right)
 			)
 		)
 		(property "Footprint" "Capacitor_THT:CP_Radial_D5.0mm_P2.00mm"
-			(at 237.1852 110.49 0)
+			(at 235.2548 102.87 0)
 			(effects
 				(font

Commit message: hella changes
Parts:
- removed D8: 80SQ045NRLG, 80SQ045NRLG:DIOAD2860W130L840D505, symbol 80SQ045NRLG:80SQ045NRLG
- added C10, C11: 100p, CAP_BF01:CAP_BF01_AVX, symbol Device:C
- added C9: 10n, CAP_BF01:CAP_BF01_AVX, symbol Device:C
- added D10: 1N4148, Diode_THT:D_DO-35_SOD27_P7.62mm_Horizontal, symbol Diode:1N4148
- added R15, R16: 9.1, Resistor_THT:R_Axial_DIN0207_L6.3mm_D2.5mm_P10.16mm_Horizontal, symbol Device:R
- added TP1, TP10, TP11, TP12, TP13, TP14, TP15, TP16, TP17, TP2, TP3, TP4, TP5, TP6, TP7, TP8, TP9: TestPoint, TestPoint:TestPoint_THTPad_D1.5mm_Drill0.7mm, symbol Connector:TestPoint
- added U4, U5: CFSH05-20L TR PBFREE, Shotky:CFSH05-20L TR PBFREE_CNS, symbol 2026-03-11_05-59-29:CFSH05-20L_TR_PBFREE
Connections:
- net +3.3V: now also TP7.1
- net +BATT: now also D10.2 (A)
- net DRV: now also TP16.1
- net GND: now also TP2.1, TP3.1; no longer U2.7 (GND)
- net GNDPWR: now also CR1.2, C10.1, C11.2, TP4.1, TP5.1, TP6.1, U4.2 (ANODE), U5.2 (ANODE)
- net PWM: now also TP12.1
- net RTN: now also TP17.1; no longer CR1.2
- net SCL: now also TP15.1
- net SDA: now also TP10.1, TP11.1, TP14.1
- net Vdrive: now also R15.2; no longer U1.8 (Vbus), U1.9 (Vin-)
- net at A1.20 (A1), R12.1, R14.2: now also TP13.1
- net at A1.30 (VIN), C2.1, L2.2: now also TP1.1
- net at J-Battery1.1, R10.1: now also R16.2, TP9.1; no longer U1.10 (Vin+)
- net at J-Battery1.2, R11.1, U3.10 (Vin+): now also TP8.1
- net at C4.1, L2.1: now also D10.1 (K)
- new net: C11.1, C9.2, R16.1, U1.10 (Vin+), U5.1 (CATHODE)
- new net: C10.2, C9.1, R15.1, U1.8 (Vbus), U1.9 (Vin-), U4.1 (CATHODE)
Other:
- moved on the sheet: A1, C2, C4, C5, C6, C7, CR1, D1, D2, D3, D4, D5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
