File: MainPCB/MAIN_PCB.kicad_sch (KiCad schematic)
At the start: 67 parts, among them U1 INA226, U2 DRV8871DDA, U3 INA226, U4 CFSH05-20L TR PBFREE, U5 CFSH05-20L TR PBFREE

Commit message: Layout
Parts:
- added C12: 0.1u, CAP_BF01:CAP_BF01_AVX, symbol Device:C
- added C13: 47u, Capacitor_THT:CP_Radial_D5.0mm_P2.00mm, symbol Device:C
- TP1: value TestPoint -> V_Buck
- TP10: value TestPoint -> I_Pump
- TP11: value TestPoint -> I_Logic
- TP12: value TestPoint -> PWM
- TP13: value TestPoint -> V_Batt
- TP14: value TestPoint -> TMP
- TP15: value TestPoint -> SCL
- TP16: value TestPoint -> DRV
- TP17: value TestPoint -> RTN
- TP2, TP3: value TestPoint -> GND
- TP4, TP5, TP6: value TestPoint -> PGND
- TP7: value TestPoint -> V_3.3
- TP8: value TestPoint -> V_Esp32
- TP9: value TestPoint -> V_Pump
Connections:
- net GND: now also C12.1, C13.2
- net at A1.30 (VIN), C2.1, L2.2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: now also C12.2, C13.1
Other:
- moved on the sheet: C2, C4, D10, L2

Commit message: 3/13
Parts:
- added C14: 10n, CAP_BF01:CAP_BF01_AVX, symbol Device:C
- added R17, R18: 9.1, Resistor_THT:R_Axial_DIN0207_L6.3mm_D2.5mm_P10.16mm_Horizontal, symbol Device:R
Connections:
- net +BATT: now also R18.2; no longer U3.8 (Vbus), U3.9 (Vin-)
- net at A1.30 (VIN), C12.2, C2.1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: no longer C13.1
- net at J-Battery1.2, R11.1, TP8.1: now also C13.1, R17.2; no longer U3.10 (Vin+)
- new net: C14.2, R17.1, U3.10 (Vin+)
- new net: C14.1, R18.1, U3.8 (Vbus), U3.9 (Vin-)
Other:
- moved on the sheet: C12, C13, R11

Commit message: Nate
Other:
- note removed: "Arduino Remote"
- note removed: "Battery"
- note removed: "Current Sensors"
- note removed: "Motor Driver"
- note removed: "Pump"
- note removed: "TMP117"
- moved on the sheet: C10, C11, C13, C14, C5, C6, C7, C9, CR1, D9, J-Battery1, J-Pump1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

Commit message: Done
Connections:
- net GND: now also J-Battery1.4; no longer J-Battery1.3
- net GNDPWR: now also J-Battery1.3; no longer J-Battery1.4
Changed lines of the file:
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@@
 	)
 	(junction
-		(at 119.38 44.45)
-		(diameter 0)
-		(color 0 0 0 0)
-	)
-	(junction
 		(at 52.07 72.39)
 		(diameter 0)
@@
 	)
 	(junction
-		(at 125.73 44.45)
-		(diameter 0)
-		(color 0 0 0 0)
-	)
-	(junction
 		(at 182.88 110.49)
 		(diameter 0)
@@
 	)
 	(junction
+		(at 125.73 44.45)
+		(diameter 0)
+		(color 0 0 0 0)
+	)
+	(junction
 		(at 100.33 177.8)
 		(diameter 0)
@@
 	(wire
 		(pts
-			(xy 119.38 44.45) (xy 125.73 44.45)
-		)
-		(stroke
-			(width 0)
-			(type default)
-		)
-	)
-	(wire
-		(pts
 			(xy 52.07 72.39) (xy 52.07 74.93)
 		)
@@
 	)
 	(symbol
+		(lib_id "power:GNDPWR")
+		(at 116.84 44.45 0)
+		(mirror y)
+		(unit 1)
+		(exclude_from_sim no)
+		(in_bom yes)
+		(on_board yes)
+		(dnp no)
+		(fields_autoplaced yes)
+		(property "Reference" "#PWR015"
+			(at 116.84 49.53 0)
+			(effects
+				(font
+					(size 1.27 1.27)
+				)
+				(hide yes)
+			)
+		)
+		(property "Value" "GNDPWR"
+			(at 116.967 48.26 0)
+			(effects
+				(font
+					(size 1.27 1.27)
+				)
+			)
+		)
+		(property "Footprint" ""
+			(at 116.84 45.72 0)
+			(effects
+				(font
+					(size 1.27 1.27)
+				)
+				(hide yes)
+			)
+		)
+		(property "Datasheet" ""
+			(at 116.84 45.72 0)
+			(effects
+				(font
+					(size 1.27 1.27)
+				)
+				(hide yes)
+			)
+		)
+		(property "Description" "Power symbol creates a global label with name \"GNDPWR\" , global ground"
+			(at 116.84 44.45 0)
+			(effects
+				(font
+					(size 1.27 1.27)
+				)
+				(hide yes)
+			)
+		)
+		(pin "1"
+		)
+		(instances
+			(project "MAIN_PCB"
+				(path "/3fbae0b3-3e6a-4fc3-bce7-3e63a917950e"
+					(reference "#PWR015")
+					(unit 1)
+				)
+			)
+		)
+	)
+	(symbol
 		(lib_id "Connector:TestPoint")
 		(at 86.36 182.88 0)
@@
 	(symbol
 		(lib_id "power:GNDPWR")
-		(at 119.38 44.45 0)
+		(at 125.73 44.45 0)
 		(mirror y)
 		(unit 1)
@@
 		(fields_autoplaced yes)
 		(property "Reference" "#PWR01"
-			(at 119.38 49.53 0)
+			(at 125.73 49.53 0)
 			(effects
 				(font
@@
 		)
 		(property "Value" "GNDPWR"
-			(at 119.507 48.26 0)
+			(at 125.857 48.26 0)
 			(effects
 				(font
@@
 		)
 		(property "Footprint" ""
-			(at 119.38 45.72 0)
+			(at 125.73 45.72 0)
 			(effects
 				(font
@@
 		)
 		(property "Datasheet" ""
-			(at 119.38 45.72 0)
+			(at 125.73 45.72 0)
 			(effects
 				(font
@@
 		)
 		(property "Description" "Power symbol creates a global label with name \"GNDPWR\" , global ground"
-			(at 119.38 44.45 0)
+			(at 125.73 44.45 0)
 			(effects
 				(font
@@
 		)
 		(instances
-			(project ""
+			(project "MAIN_PCB"
 				(path "/3fbae0b3-3e6a-4fc3-bce7-3e63a917950e"
 					(reference "#PWR01")
@@
 	)
 	(symbol
+		(lib_id "power:GND")
+		(at 119.38 44.45 0)
+		(mirror y)
+		(unit 1)
+		(exclude_from_sim no)
+		(in_bom yes)
+		(on_board yes)
+		(dnp no)
+		(fields_autoplaced yes)
+		(property "Reference" "#PWR047"
+			(at 119.38 50.8 0)
+			(effects
+				(font
+					(size 1.27 1.27)
+				)
+				(hide yes)
+			)
+		)
+		(property "Value" "GND"
+			(at 119.38 49.53 0)
+			(effects
+				(font
+					(size 1.27 1.27)
+				)
+			)
+		)
+		(property "Footprint" ""
+			(at 119.38 44.45 0)
+			(effects
+				(font
+					(size 1.27 1.27)
+				)
+				(hide yes)
+			)
+		)
+		(property "Datasheet" ""
+			(at 119.38 44.45 0)
+			(effects
+				(font
+					(size 1.27 1.27)
+				)
+				(hide yes)
+			)
+		)
+		(property "Description" "Power symbol creates a global label with name \"GND\" , ground"
+			(at 119.38 44.45 0)
+			(effects
+				(font
+					(size 1.27 1.27)
+				)
+				(hide yes)
+			)
+		)
+		(pin "1"
+		)
+		(instances
+			(project "MAIN_PCB"
+				(path "/3fbae0b3-3e6a-4fc3-bce7-3e63a917950e"
+					(reference "#PWR047")
+					(unit 1)
+				)
+			)
+		)
+	)
+	(symbol
 		(lib_id "power:+3.3V")
 		(at 170.18 71.12 270)
@@
 					(unit 1)
 				)
-			)
-		)
-	)
-	(symbol
-		(lib_id "power:GND")
-		(at 116.84 44.45 0)
-		(mirror y)
-		(unit 1)
-		(exclude_from_sim no)
-		(in_bom yes)
-		(on_board yes)
-		(dnp no)
-		(fields_autoplaced yes)
-		(property "Reference" "#PWR015"
-			(at 116.84 50.8 0)
-			(effects
-				(font
-					(size 1.27 1.27)
-				)
-				(hide yes)
-			)
-		)
-		(property "Value" "GND"
-			(at 116.8399 48.26 90)
-			(effects
-				(font
-					(size 1.27 1.27)
-				)
-				(justify right)
-			)
-		)
-		(property "Footprint" ""
-			(at 116.84 44.45 0)
-			(effects
-				(font
-					(size 1.27 1.27)
-				)
-				(hide yes)
-			)
-		)
-		(property "Datasheet" ""
-			(at 116.84 44.45 0)
-			(effects
-				(font
-					(size 1.27 1.27)
-				)
-				(hide yes)
-			)
-		)
-		(property "Description" "Power symbol creates a global label with name \"GND\" , ground"
-			(at 116.84 44.45 0)
-			(effects
-				(font
-					(size 1.27 1.27)
-				)
-				(hide yes)
-			)
-		)
-		(pin "1"
-		)
-		(instances
-			(project "MAIN_PCB"
-				(path "/3fbae0b3-3e6a-4fc3-bce7-3e63a917950e"
-					(reference "#PWR015")
-					(unit 1)
-				)
