File: MainPCB/MAIN_PCB.kicad_pcb (KiCad board)
At the start: 2 copper layers, 1 part

Commit message: c
Parts:
- added U1: DRV8871DDA, Package_SO:Texas_HTSOP-8-1EP_3.9x4.9mm_P1.27mm_EP2.95x4.9mm_Mask2.4x3.1mm_ThermalVias, F.Cu at (212.1, 75.6)

Commit message: a
Parts:
- removed A1: Arduino_Nano_ESP32, Module:Arduino_Nano
- added A2: Arduino_Nano_ESP32, Module:Arduino_Nano, F.Cu at (183.9, 79.0)
- added C1: 10uF, Capacitor_SMD:C_1206_3216Metric, F.Cu at (223.1, 76.1)
- added C2: 10uF, Capacitor_SMD:C_1206_3216Metric, F.Cu at (223.1, 79.4)
- added C3: 0.1uF, Capacitor_SMD:C_1206_3216Metric, F.Cu at (223.1, 82.8)
- added D1: LED Auto, LED_THT:LED_D3.0mm, F.Cu at (213.6, 102.3)
- added D2: BAT3, LED_THT:LED_D3.0mm, F.Cu at (213.6, 107.8)
- added D3: BAT2, LED_THT:LED_D3.0mm, F.Cu at (213.6, 113.3)
- added D4: BAT1, LED_THT:LED_D3.0mm, F.Cu at (213.6, 118.7)
- added D5: MAN 3, LED_THT:LED_D3.0mm, F.Cu at (219.5, 102.3)
- added D6: MAN 2, LED_THT:LED_D3.0mm, F.Cu at (219.5, 107.8)
- added D7: MAN 1, LED_THT:LED_D3.0mm, F.Cu at (219.5, 113.3)
- added D8: US1M, Diode_SMD:D_SMA, F.Cu at (224.4, 86.7)
- added J4: Conn_01x04_Socket, Connector_PinHeader_2.54mm:PinHeader_1x04_P2.54mm_Vertical, F.Cu at (226.0, 101.9)
- added J7: Screw_Terminal_01x02, TerminalBlock_4Ucon:TerminalBlock_4Ucon_1x02_P3.50mm_Horizontal, F.Cu at (204.3, 115.3)
- added R1: R, Resistor_THT:R_Axial_DIN0207_L6.3mm_D2.5mm_P7.62mm_Horizontal, F.Cu at (202.7, 76.4)
- added R2: R, Resistor_THT:R_Axial_DIN0207_L6.3mm_D2.5mm_P7.62mm_Horizontal, F.Cu at (202.7, 80.5)
- added R3: R, Resistor_THT:R_Axial_DIN0207_L6.3mm_D2.5mm_P7.62mm_Horizontal, F.Cu at (202.7, 84.5)
- added R4: R, Resistor_THT:R_Axial_DIN0207_L6.3mm_D2.5mm_P7.62mm_Horizontal, F.Cu at (202.7, 88.6)
- added R5: R, Resistor_THT:R_Axial_DIN0207_L6.3mm_D2.5mm_P7.62mm_Horizontal, F.Cu at (202.7, 92.6)
- added R6: R, Resistor_THT:R_Axial_DIN0207_L6.3mm_D2.5mm_P7.62mm_Horizontal, F.Cu at (202.7, 96.7)
- added R7: R, Resistor_THT:R_Axial_DIN0207_L6.3mm_D2.5mm_P7.62mm_Horizontal, F.Cu at (202.7, 100.7)
- added R8: R, Resistor_THT:R_Axial_DIN0207_L6.3mm_D2.5mm_P7.62mm_Horizontal, F.Cu at (202.7, 104.8)
- added R9: R, Resistor_THT:R_Axial_DIN0207_L6.3mm_D2.5mm_P7.62mm_Horizontal, F.Cu at (202.7, 108.8)
- added S1: SG06280N, SG06280N:SW_SG06280N, F.Cu at (216.1, 78.6)
- added S2: SG06280N, SG06280N:SW_SG06280N, F.Cu at (216.1, 87.0)
- added S3: SG06280N, SG06280N:SW_SG06280N, F.Cu at (216.1, 95.4)
- U1: value DRV8871DDA -> INA226; footprint Package_SO:Texas_HTSOP-8-1EP_3.9x4.9mm_P1.27mm_EP2.95x4.9mm_Mask2.4x3.1mm_ThermalVias -> Package_SO:VSSOP-10_3x3mm_P0.5mm
- moved U1 19.7 mm to (224.0, 91.3)
Connections:
- U1 pad 1: Net-(U1-GND-Pad1) -> unconnected-(U1-A1-Pad1)
- U1 pad 4: unconnected-(U1-ILIM-Pad4) -> SDA
- U1 pad 5: unconnected-(U1-VM-Pad5) -> SCL
- U1 pad 6: unconnected-(U1-OUT1-Pad6) -> +3.3V
- U1 pad 7: Net-(U1-GND-Pad1) -> GND
- U1 pad 9: Net-(U1-GND-Pad1) -> unconnected-(U1-Vin--Pad9)

Commit message: a
Parts:
- S1, S2, S3: value SG06280N -> TL3315NF250Q; footprint SG06280N:SW_SG06280N -> TL3315NF250Q:SW_TL3315NF250Q
- moved S1 18.7 mm to (234.3, 83.0)
- moved S2 18.3 mm to (234.3, 89.1)
- moved S3 18.2 mm to (234.3, 95.2)
Connections:
- S1 pad 1: GND -> Net-(A2-A2)
- S1 pad 2: Net-(A2-D2) -> Net-(A2-A2)
- S2 pad 2: GND -> Net-(A2-A3)
- S3 pad 1: Net-(A2-A2) -> GND

Commit message: 2/13
Parts:
- removed J4: Conn_01x04_Socket, Connector_PinHeader_2.54mm:PinHeader_1x04_P2.54mm_Vertical
- removed J7: Screw_Terminal_01x02, TerminalBlock_4Ucon:TerminalBlock_4Ucon_1x02_P3.50mm_Horizontal
- added J1: SS-12800-009, SS_12800_009:STEWART_SS-12800-009, F.Cu at (182.1, 129.5)
- added J2: SS-12800-009, SS_12800_009:STEWART_SS-12800-009, F.Cu at (203.4, 129.5)
- added J5: SS-12800-009, SS_12800_009:STEWART_SS-12800-009, F.Cu at (224.8, 129.5)
- added JP1: SolderJumper_2_Open, Jumper:SolderJumper-2_P1.3mm_Open_TrianglePad1.0x1.5mm, F.Cu at (243.6, 109.2)
- added JP2: SolderJumper_2_Open, Jumper:SolderJumper-2_P1.3mm_Open_TrianglePad1.0x1.5mm, F.Cu at (243.6, 112.7)
- added JP3: SolderJumper_2_Open, Jumper:SolderJumper-2_P1.3mm_Open_TrianglePad1.0x1.5mm, F.Cu at (243.6, 116.3)
- added JP4: SolderJumper_2_Open, Jumper:SolderJumper-2_P1.3mm_Open_TrianglePad1.0x1.5mm, F.Cu at (243.6, 119.8)
- added JP5: SolderJumper_2_Open, Jumper:SolderJumper-2_P1.3mm_Open_TrianglePad1.0x1.5mm, F.Cu at (243.6, 123.4)
- added JP6: SolderJumper_2_Open, Jumper:SolderJumper-2_P1.3mm_Open_TrianglePad1.0x1.5mm, F.Cu at (243.6, 126.9)
- added R10: 68m, Resistor_SMD:R_1206_3216Metric, F.Cu at (258.0, 118.4)
- added R11: 100m, Resistor_SMD:R_1206_3216Metric, F.Cu at (258.0, 121.7)
- added R12: 120m, Resistor_SMD:R_1206_3216Metric, F.Cu at (258.0, 125.0)
- added U2: DRV8871DDA, Package_SO:Texas_HTSOP-8-1EP_3.9x4.9mm_P1.27mm_EP2.95x4.9mm_Mask2.4x3.1mm_ThermalVias, F.Cu at (250.5, 120.1)
- added U4: XTPS55285VALR, footprints:VAL0015A-MFG, F.Cu at (249.0, 125.6)
- D1, D2, D3, D4, D5, D6, D7: footprint LED_THT:LED_D3.0mm -> LED_SMD:LED_1206_3216Metric
- R1, R2, R3, R4, R5, R6, R7: value R -> 220; footprint Resistor_THT:R_Axial_DIN0207_L6.3mm_D2.5mm_P7.62mm_Horizontal -> Resistor_SMD:R_1206_3216Metric
- R8, R9: footprint Resistor_THT:R_Axial_DIN0207_L6.3mm_D2.5mm_P7.62mm_Horizontal -> Resistor_SMD:R_1206_3216Metric
- moved S1 18.5 mm to (216.2, 78.8)
- moved S2 18.5 mm to (216.2, 84.9)
- moved S3 18.5 mm to (216.2, 91.0)
Connections:
- U1 pad 1: unconnected-(U1-A1-Pad1) -> GND
- U1 pad 10: unconnected-(U1-Vin+-Pad10) -> Net-(JP2-B)
- U1 pad 2: unconnected-(U1-A0-Pad2) -> GND
- U1 pad 8: unconnected-(U1-Vbus-Pad8) -> Net-(JP1-A)
- U1 pad 9: unconnected-(U1-Vin--Pad9) -> Net-(JP1-A)

Commit message: a
Parts:
- added J4: Conn_01x04_Socket, Connector_PinHeader_2.54mm:PinHeader_1x04_P2.54mm_Vertical, F.Cu at (175.0, 127.4)
- added J6: 853-002-213R00Y, SS_12800_009:853-002-213R00Y, F.Cu at (235.7, 82.8)
- added J7: 853-002-213R00Y, SS_12800_009:853-002-213R00Y, F.Cu at (254.4, 82.8)

Commit message: a
Parts:
- removed J1, J2, J5: SS-12800-009, SS_12800_009:STEWART_SS-12800-009
- removed J4: Conn_01x04_Socket, Connector_PinHeader_2.54mm:PinHeader_1x04_P2.54mm_Vertical
- removed J6, J7: 853-002-213R00Y, SS_12800_009:853-002-213R00Y
- removed JP1, JP2, JP3, JP4, JP5, JP6: SolderJumper_2_Open, Jumper:SolderJumper-2_P1.3mm_Open_TrianglePad1.0x1.5mm
- removed R11: 100m, Resistor_SMD:R_1206_3216Metric
- removed R12: 120m, Resistor_SMD:R_1206_3216Metric
- removed U4: XTPS55285VALR, footprints:VAL0015A-MFG
- added C4: BQ014E0473J, CAP_BF01:CAP_BF01_AVX, F.Cu at (128.9, 82.7)
- added D9: US1M, Diode_SMD:D_SMA, F.Cu at (127.2, 112.0)
- added J-Battery1: 861-004-213R00Y, 861.preety:861-004-213R00Y, F.Cu at (109.3, 90.9)
- added J-Pump1: 861-004-213R00Y, 861.preety:861-004-213R00Y, F.Cu at (99.5, 119.7)
- added J-TMP1: 861-004-213R00Y, 861.preety:861-004-213R00Y, F.Cu at (85.3, 90.8)
- added L2: LQH44PH220MPRL, IND_LQH44PN:IND_LQH44PN_PR_MUR-L, F.Cu at (132.9, 75.5)
- added R13: 32k, Resistor_SMD:R_1206_3216Metric, F.Cu at (128.0, 104.5)
- C2: value 10uF -> BQ014E0473J; footprint Capacitor_SMD:C_1206_3216Metric -> CAP_BF01:CAP_BF01_AVX
- R10: value 68m -> 100m
- R8, R9: value R -> 2.2k
- moved R9 133.4 mm to (70.5, 91.3)
- moved R8 133.3 mm to (70.5, 88.0)
- moved R10 130.9 mm to (130.4, 89.3), turned to 180 degrees
- moved U2 123.3 mm to (127.2, 120.7), turned to 90 degrees
- moved D7 121.8 mm to (97.9, 119.9), turned to -90 degrees
- moved D6 118.9 mm to (101.2, 119.9), turned to -90 degrees
- moved S3 117.7 mm to (100.3, 111.5), turned to -90 degrees
- moved D5 116.2 mm to (104.6, 119.9), turned to -90 degrees
- moved S2 112.9 mm to (106.5, 111.5), turned to -90 degrees
- moved S1 108.6 mm to (112.7, 111.5), turned to -90 degrees
- moved A2 108.3 mm to (78.5, 104.0), turned to 90 degrees
- moved R7 108.1 mm to (97.6, 125.6), turned to -90 degrees
- moved D4 105.6 mm to (108.0, 119.9), turned to -90 degrees
- moved R6 105.1 mm to (101.7, 125.5), turned to -90 degrees
- moved R5 103.1 mm to (105.0, 125.5), turned to -90 degrees
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Connections:
- A2 pad 20: unconnected-(A2-A1-Pad20) -> PWM
- A2 pad 25: IN1 -> unconnected-(A2-A6-Pad25)
- A2 pad 26: IN2 -> unconnected-(A2-A7-Pad26)
- C2 pad 1: GND -> Net-(A2-VIN)
- C2 pad 2: Net-(A2-VIN) -> GND
- D8 pad 1: Net-(A2-VIN) -> Net-(D8-K)
- D8 pad 2: Net-(D8-A) -> +BATT
- R10 pad 1: Net-(JP2-A) -> +BATT
- R10 pad 2: Net-(JP1-B) -> Vdrive
- U1 pad 10: Net-(JP2-B) -> +BATT
- U1 pad 8: Net-(JP1-A) -> Vdrive
- U1 pad 9: Net-(JP1-A) -> Vdrive
- U2 pad 1: Net-(U2-GND-Pad1) -> GND
- U2 pad 2: unconnected-(U2-IN2-Pad2) -> GND
- U2 pad 3: unconnected-(U2-IN1-Pad3) -> PWM
- U2 pad 4: unconnected-(U2-ILIM-Pad4) -> Net-(U2-ILIM)
- U2 pad 5: unconnected-(U2-VM-Pad5) -> Vdrive
- U2 pad 6: unconnected-(U2-OUT1-Pad6) -> DRV
- U2 pad 7: Net-(U2-GND-Pad1) -> GND
- U2 pad 8: unconnected-(U2-OUT2-Pad8) -> RTN
- U2 pad 9: Net-(U2-GND-Pad1) -> GNDPWR
Routing:
- net GND: track 0.00 -> 219.4 mm, vias 0 -> 1
- net GNDPWR: track 0.00 -> 103.1 mm, vias 0 -> 1
- net DRV: track 0.00 -> 71.9 mm
- net +3.3V: track 0.00 -> 50.1 mm
- net RTN: track 0.00 -> 45.5 mm
Other:
- board outline added: 75 x 70.5 mm

Commit message: Nate
Parts:
- removed A2: Arduino_Nano_ESP32, Module:Arduino_Nano
- added A1: Arduino_Nano_ESP32, Module:Arduino_Nano, F.Cu at (78.3, 104.0)
Connections:
- D9 pad 2: GND -> GNDPWR
- J-Battery1 pad 1: +BATT -> Net-(U1-Vin+)
- J-Pump1 pad 3: GND -> GNDPWR
- J-Pump1 pad 4: GND -> GNDPWR
- R10 pad 1: +BATT -> Net-(U1-Vin+)
- U1 pad 10: +BATT -> Net-(U1-Vin+)
- U2 pad 9: GNDPWR -> GND

Commit message: Nate
Parts:
- added R1: 56, Resistor_THT:R_Axial_DIN0207_L6.3mm_D2.5mm_P7.62mm_Horizontal, F.Cu at (96.8, 139.8)
- added R2: 56, Resistor_THT:R_Axial_DIN0207_L6.3mm_D2.5mm_P7.62mm_Horizontal, F.Cu at (100.9, 139.8)
- added R3: 56, Resistor_THT:R_Axial_DIN0207_L6.3mm_D2.5mm_P7.62mm_Horizontal, F.Cu at (105.0, 139.8)
- added R4: 56, Resistor_THT:R_Axial_DIN0207_L6.3mm_D2.5mm_P7.62mm_Horizontal, F.Cu at (109.0, 139.8)
- added R5: 56, Resistor_THT:R_Axial_DIN0207_L6.3mm_D2.5mm_P7.62mm_Horizontal, F.Cu at (113.0, 139.8)
- added R6: 56, Resistor_THT:R_Axial_DIN0207_L6.3mm_D2.5mm_P7.62mm_Horizontal, F.Cu at (117.1, 139.8)
- added R7: 56, Resistor_THT:R_Axial_DIN0207_L6.3mm_D2.5mm_P7.62mm_Horizontal, F.Cu at (121.2, 139.8)
- R13, R8, R9: footprint Resistor_SMD:R_1206_3216Metric -> Resistor_THT:R_Axial_DIN0207_L6.3mm_D2.5mm_P7.62mm_Horizontal
