File: MainPCB/MAIN_PCB.kicad_pcb (KiCad board)
At the start: 2 copper layers, 75 x 70.5 mm, 41 parts, among them U1 INA226, U2 DRV8871DDA

Commit message: 3/8
Parts:
- removed J-TMP1: 861-004-213R00Y, 861.preety:861-004-213R00Y
- removed the R1 at (118.2, 125.5)
- removed the R1 at (96.8, 139.8)
- removed the R2 at (100.9, 139.8)
- removed the R2 at (114.9, 125.5)
- removed the R3 at (105.0, 139.8)
- removed the R3 at (111.6, 125.5)
- removed the R4 at (108.3, 125.5)
- removed the R4 at (109.0, 139.8)
- removed the R5 at (105.0, 125.5)
- removed the R5 at (113.0, 139.8)
- removed the R6 at (117.1, 139.8)
- removed the R6 at (101.7, 125.5)
- removed the R7 at (121.2, 139.8)
- removed the R7 at (97.6, 125.6)
- added C5: 0.1u, CAP_BF01:CAP_BF01_AVX, F.Cu at (83.9, 103.9)
- added C6: 100u, Capacitor_THT:CP_Radial_D5.0mm_P2.00mm, F.Cu at (155.2, 114.0)
- added C7: 10u, Capacitor_THT:CP_Radial_D5.0mm_P2.00mm, F.Cu at (155.2, 120.5)
- added CR1: SA15CA, DO-204AC_SA:DO-204AC_SA, F.Cu at (177.1, 106.8)
- added J-TMP117: 861-004-213R00Y, 861.preety:861-004-213R00Y, F.Cu at (103.2, 143.6)
- added R1: 56, Resistor_THT:R_Axial_DIN0207_L6.3mm_D2.5mm_P7.62mm_Horizontal, F.Cu at (136.8, 92.6)
- added R2: 56, Resistor_THT:R_Axial_DIN0207_L6.3mm_D2.5mm_P7.62mm_Horizontal, F.Cu at (136.8, 96.6)
- added R3: 56, Resistor_THT:R_Axial_DIN0207_L6.3mm_D2.5mm_P7.62mm_Horizontal, F.Cu at (136.8, 100.7)
- added R4: 56, Resistor_THT:R_Axial_DIN0207_L6.3mm_D2.5mm_P7.62mm_Horizontal, F.Cu at (136.8, 104.7)
- added R5: 56, Resistor_THT:R_Axial_DIN0207_L6.3mm_D2.5mm_P7.62mm_Horizontal, F.Cu at (136.8, 108.8)
- added R6: 56, Resistor_THT:R_Axial_DIN0207_L6.3mm_D2.5mm_P7.62mm_Horizontal, F.Cu at (136.8, 112.8)
- added R7: 56, Resistor_THT:R_Axial_DIN0207_L6.3mm_D2.5mm_P7.62mm_Horizontal, F.Cu at (136.8, 116.9)
- C1: footprint Capacitor_SMD:C_1206_3216Metric -> Capacitor_THT:CP_Radial_D5.0mm_P2.00mm
- C3: footprint Capacitor_SMD:C_1206_3216Metric -> CAP_BF01:CAP_BF01_AVX
- D1, D2, D3, D4, D5, D6, D7: footprint LED_SMD:LED_1206_3216Metric -> LED_THT:LED_Oval_W5.2mm_H3.8mm
- D8, D9: value US1M -> 80SQ045NRLG; footprint Diode_SMD:D_SMA -> 80SQ045NRLG:DIOAD2860W130L840D505
- L2: footprint IND_LQH44PN:IND_LQH44PN_PR_MUR-L -> IND_LQH44PN:IND_LQH44PN_PR_MUR
- moved D8 88.3 mm to (119.5, 163.5), turned to 90 degrees
- moved J-Pump1 84.6 mm to (149.0, 51.1), turned to 0 degrees
- moved C2 80.9 mm to (107.4, 146.5)
- moved R9 74.4 mm to (136.8, 125.0)
- moved R8 74.0 mm to (136.8, 120.9)
- moved L2 69.4 mm to (109.9, 141.0), turned to -90 degrees
- moved J-Battery1 66.9 mm to (80.2, 151.1), turned to 0 degrees
- moved R10 65.7 mm to (179.0, 133.5), turned to 0 degrees
- moved S3 64.5 mm to (163.4, 124.7), turned to 0 degrees
- moved C1 60.3 mm to (85.5, 137.5), turned to 90 degrees
- moved S2 57.4 mm to (163.4, 118.6), turned to 0 degrees
- moved C4 57.0 mm to (107.4, 135.5)
- moved U1 55.5 mm to (170.5, 134.9), turned to 0 degrees
- moved C3 53.5 mm to (83.9, 95.6)
- moved S1 50.8 mm to (163.4, 112.4), turned to 0 degrees
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Routing:
- net GND: track 219.4 -> 0.00 mm, vias 1 -> 0
- net GNDPWR: track 103.1 -> 0.00 mm, vias 1 -> 0
- net DRV: track 71.9 -> 0.00 mm
- net +3.3V: track 50.1 -> 0.00 mm
- net RTN: track 45.5 -> 0.00 mm
Other:
- board size 75 x 70.5 mm -> 1.2 x 1.2 mm

Commit message: Nate
Parts:
- moved S1 142.0 mm to (274.8, 24.2)
- moved S2 142.0 mm to (274.8, 30.4)
- moved S3 142.0 mm to (274.8, 36.5)
- moved C5 88.9 mm to (170.4, 83.3)
- moved D8 80.3 mm to (173.5, 104.1), turned to -90 degrees
- moved D7 69.3 mm to (128.6, 59.6), turned to -90 degrees
- moved R7 68.6 mm to (137.8, 48.3), turned to -90 degrees
- moved J-Battery1 65.8 mm to (131.0, 109.3)
- moved A1 65.5 mm to (163.6, 67.9)
- moved C1 65.5 mm to (130.6, 89.9)
- moved C2 65.5 mm to (152.4, 98.9)
- moved C4 65.5 mm to (152.5, 87.9)
- moved R6 64.7 mm to (141.9, 48.3), turned to -90 degrees
- moved L2 63.6 mm to (152.0, 93.3)
- moved D6 62.6 mm to (134.1, 59.6), turned to -90 degrees
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
Commit message: Nate
Routing:
- net +3.3V: track 0.00 -> 25.8 mm
Changed lines of the file:
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@@
 		)
+	)
+	(segment
+		(start 130.53 87.87)
+		(end 130.55 87.89)
+		(width 0.2)
+		(layer "F.Cu")
+		(net 1)
+	)
+	(segment
+		(start 149.458824 107.39)
+		(end 149.726 107.122824)
+		(width 0.2)
+		(layer "F.Cu")
+		(net 1)
+	)
+	(segment
+		(start 149.726 89.526)
+		(end 148.09 87.89)
+		(width 0.2)
+		(layer "F.Cu")
+		(net 1)
+	)
+	(segment
+		(start 148.7 107.39)
+		(end 149.458824 107.39)
+		(width 0.2)
+		(layer "F.Cu")
+		(net 1)
+	)
+	(segment
+		(start 130.53 83.13)
+		(end 130.53 87.87)
+		(width 0.2)
+		(layer "F.Cu")
+		(net 1)
+	)
+	(segment
+		(start 149.726 107.122824)
+		(end 149.726 89.526)
+		(width 0.2)
+		(layer "F.Cu")
+		(net 1)
+	)
+	(segment
+		(start 130.55 89.89)
+		(end 130.66 90)
+		(width 0.2)
+		(layer "F.Cu")
+		(net 4)
 	)
 	(embedded_fonts no)

Commit message: nate
Parts:
- added C8: 0.1uF, CAP_BF01:CAP_BF01_AVX, F.Cu at (171.0, 93.5)
- added R11: Shunt, Resistor_SMD:R_1206_3216Metric, F.Cu at (175.5, 96.5)
- added R12: 100k, Resistor_THT:R_Axial_DIN0207_L6.3mm_D2.5mm_P10.16mm_Horizontal, F.Cu at (173.4, 64.7)
- added R14: 390k, Resistor_THT:R_Axial_DIN0207_L6.3mm_D2.5mm_P10.16mm_Horizontal, F.Cu at (177.5, 54.5)
- added U3: INA226, Package_SO:VSSOP-10_3x3mm_P0.5mm, F.Cu at (176.0, 90.2)
- R1, R13, R2, R3, R4, R5, R6, R7, R8, R9: footprint Resistor_THT:R_Axial_DIN0207_L6.3mm_D2.5mm_P7.62mm_Horizontal -> Resistor_THT:R_Axial_DIN0207_L6.3mm_D2.5mm_P10.16mm_Horizontal
- R10: value 100m -> Shunt
- moved S1 142.1 mm to (137.8, 62.0), turned to 180 degrees
- moved S2 139.4 mm to (137.8, 55.9), turned to 180 degrees
- moved S3 137.6 mm to (137.8, 49.8), turned to 180 degrees
- moved J-Battery1 78.8 mm to (199.8, 70.8), turned to 180 degrees
- moved D8 50.1 mm to (184.5, 55.2)
- moved C6 45.5 mm to (146.5, 109.0), turned to 90 degrees
- moved D7 45.4 mm to (172.5, 48.0)
- moved C7 43.5 mm to (140.0, 107.3), turned to 90 degrees
- moved C5 42.5 mm to (134.3, 105.7), turned to 90 degrees
- moved U2 38.9 mm to (143.0, 98.5), turned to -90 degrees
- moved J-Pump1 36.8 mm to (176.9, 95.4), turned to 0 degrees
- moved D6 34.9 mm to (167.0, 48.0)
- moved C2 34.9 mm to (185.5, 88.0), turned to 180 degrees
- moved C4 34.8 mm to (185.5, 99.0), turned to 180 degrees
- moved L2 31.2 mm to (183.2, 93.6), turned to 90 degrees
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Connections:
- A1 pad 19: unconnected-(A1-A0-Pad19) -> PWM
- A1 pad 20: PWM -> Net-(A1-A1)
- C5 pad 1: GND -> GNDPWR
- C6 pad 1: GND -> GNDPWR
- C7 pad 1: GND -> GNDPWR
- J-Battery1 pad 2: +BATT -> Net-(U3-Vin+)
Routing:
- net +3.3V: track 25.8 -> 130.4 mm, vias 0 -> 1
- net Vdrive: track 0.00 -> 91.7 mm, vias 0 -> 1
- net SCL: track 0.00 -> 75.3 mm, vias 0 -> 1
- net Net-(U1-Vin+): track 0.00 -> 70.8 mm, vias 0 -> 1
- net +BATT: track 0.00 -> 69.6 mm
- net Net-(U3-Vin+): track 0.00 -> 58.7 mm, vias 0 -> 1
- net Net-(A1-A1): track 0.00 -> 56.3 mm, vias 0 -> 1
- net Net-(A1-D2): track 0.00 -> 52.1 mm, vias 0 -> 1
- net Net-(D8-K): track 0.00 -> 50.9 mm, vias 0 -> 1
- net DRV: track 0.00 -> 40.8 mm
- net Net-(A1-A3): track 0.00 -> 38.4 mm, vias 0 -> 1
- net RTN: track 0.00 -> 38.4 mm
- net Net-(A1-A2): track 0.00 -> 32.8 mm, vias 0 -> 1
- net SDA: track 0.00 -> 28.1 mm
- net Net-(A1-VIN): track 0.00 -> 16.7 mm, vias 0 -> 1
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
Commit message: DRV8871
Parts:
- moved R11 1.10 mm to (175.4, 95.4)
- moved C8 1.00 mm to (171.0, 94.5)
- moved L2 0.63 mm to (183.6, 93.0), turned to 0 degrees
Connections:
- C1 pad 1: GND -> +3.3V
- C1 pad 2: +3.3V -> GND
- C5 pad 1: GNDPWR -> GND
- C6 pad 1: GNDPWR -> Vdrive
- C6 pad 2: Vdrive -> GNDPWR
- C7 pad 1: GNDPWR -> Vdrive
- C7 pad 2: Vdrive -> GND
Routing:
- net SDA: track 28.1 -> 94.6 mm, vias 0 -> 1
- net +3.3V: track 130.4 -> 116.0 mm
- net Net-(U1-Vin+): track 70.8 -> 75.3 mm
- net Net-(D8-K): track 50.9 -> 55.0 mm
- net Net-(U3-Vin+): track 58.7 -> 61.0 mm
- net Net-(A1-VIN): track 16.7 -> 18.0 mm
- net SCL: track 75.3 -> 74.2 mm
- net Vdrive: track 91.7 -> 90.8 mm
- added copper zone on B.Cu, net GNDPWR
Other:
- board size 1.2 x 1.2 mm -> 81.5 x 76.5 mm

Commit message: hella changes
Parts:
- removed D8: 80SQ045NRLG, 80SQ045NRLG:DIOAD2860W130L840D505
- added C10: 100p, CAP_BF01:CAP_BF01_AVX, F.Cu at (158.9, 130.9)
- added C11: 100p, CAP_BF01:CAP_BF01_AVX, F.Cu at (158.9, 135.0)
- added C9: 10n, CAP_BF01:CAP_BF01_AVX, F.Cu at (158.9, 126.7)
- added D10: 1N4148, Diode_THT:D_DO-35_SOD27_P7.62mm_Horizontal, F.Cu at (174.9, 138.9)
- added R15: 9.1, Resistor_THT:R_Axial_DIN0207_L6.3mm_D2.5mm_P10.16mm_Horizontal, F.Cu at (121.9, 184.1)
- added R16: 9.1, Resistor_THT:R_Axial_DIN0207_L6.3mm_D2.5mm_P10.16mm_Horizontal, F.Cu at (121.9, 188.2)
- added TP1: TestPoint, TestPoint:TestPoint_THTPad_D1.5mm_Drill0.7mm, F.Cu at (68.5, 110.0)
- added TP10: TestPoint, TestPoint:TestPoint_THTPad_D1.5mm_Drill0.7mm, F.Cu at (72.0, 120.7)
- added TP11: TestPoint, TestPoint:TestPoint_THTPad_D1.5mm_Drill0.7mm, F.Cu at (72.0, 124.2)
- added TP12: TestPoint, TestPoint:TestPoint_THTPad_D1.5mm_Drill0.7mm, F.Cu at (72.0, 127.8)
- added TP13: TestPoint, TestPoint:TestPoint_THTPad_D1.5mm_Drill0.7mm, F.Cu at (75.6, 110.0)
- added TP14: TestPoint, TestPoint:TestPoint_THTPad_D1.5mm_Drill0.7mm, F.Cu at (75.6, 113.5)
- added TP15: TestPoint, TestPoint:TestPoint_THTPad_D1.5mm_Drill0.7mm, F.Cu at (75.6, 117.1)
- added TP16: TestPoint, TestPoint:TestPoint_THTPad_D1.5mm_Drill0.7mm, F.Cu at (75.6, 120.7)
- added TP17: TestPoint, TestPoint:TestPoint_THTPad_D1.5mm_Drill0.7mm, F.Cu at (75.6, 124.2)
- added TP2: TestPoint, TestPoint:TestPoint_THTPad_D1.5mm_Drill0.7mm, F.Cu at (68.5, 113.5)
- added TP3: TestPoint, TestPoint:TestPoint_THTPad_D1.5mm_Drill0.7mm, F.Cu at (68.5, 117.1)
- added TP4: TestPoint, TestPoint:TestPoint_THTPad_D1.5mm_Drill0.7mm, F.Cu at (68.5, 120.7)
- added TP5: TestPoint, TestPoint:TestPoint_THTPad_D1.5mm_Drill0.7mm, F.Cu at (68.5, 124.2)
- added TP6: TestPoint, TestPoint:TestPoint_THTPad_D1.5mm_Drill0.7mm, F.Cu at (68.5, 127.8)
- added TP7: TestPoint, TestPoint:TestPoint_THTPad_D1.5mm_Drill0.7mm, F.Cu at (72.0, 110.0)
- added TP8: TestPoint, TestPoint:TestPoint_THTPad_D1.5mm_Drill0.7mm, F.Cu at (72.0, 113.5)
- added TP9: TestPoint, TestPoint:TestPoint_THTPad_D1.5mm_Drill0.7mm, F.Cu at (72.0, 117.1)
- added U4: CFSH05-20L TR PBFREE, Shotky:CFSH05-20L TR PBFREE_CNS, F.Cu at (184.1, 154.3)
- added U5: CFSH05-20L TR PBFREE, Shotky:CFSH05-20L TR PBFREE_CNS, F.Cu at (184.1, 156.6)
- moved J-Battery1 177.9 mm to (23.8, 44.9), turned to 0 degrees
- moved J-Pump1 140.3 mm to (46.0, 44.9)
- moved R14 137.3 mm to (121.9, 180.1), turned to 0 degrees
- moved J-TMP117 131.1 mm to (68.2, 44.9), turned to 0 degrees
- moved R12 119.0 mm to (121.9, 171.9), turned to 0 degrees
- moved D7 110.9 mm to (111.0, 140.3), turned to 0 degrees
- moved S3 107.7 mm to (169.9, 152.5), turned to 0 degrees
- moved D6 103.3 mm to (111.0, 134.8), turned to 0 degrees
- moved S2 96.0 mm to (169.9, 146.4), turned to 0 degrees
- moved D5 95.8 mm to (111.0, 129.4), turned to 0 degrees
- moved R13 90.0 mm to (121.9, 176.0), turned to 0 degrees
- moved D1 89.6 mm to (111.0, 107.5), turned to 0 degrees
- moved D4 88.2 mm to (111.0, 123.9), turned to 0 degrees
- moved R9 85.6 mm to (121.9, 167.9), turned to 0 degrees
- moved R8 85.6 mm to (121.9, 163.8), turned to 0 degrees
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Connections:
- CR1 pad 2: RTN -> GNDPWR
- J-Battery1 pad 1: Net-(U1-Vin+) -> Net-(J-Battery1-Pad1)
- R10 pad 1: Net-(U1-Vin+) -> Net-(J-Battery1-Pad1)
- U1 pad 8: Vdrive -> Net-(U1-Vbus)
- U1 pad 9: Vdrive -> Net-(U1-Vbus)
- U2 pad 7: GND -> GNDPWR
Routing:
- net +3.3V: track 116.0 -> 0.00 mm, vias 1 -> 0
- net SDA: track 94.6 -> 0.00 mm, vias 1 -> 0
- net Vdrive: track 90.8 -> 0.00 mm, vias 1 -> 0
- net Net-(U1-Vin+): track 75.3 -> 0.00 mm, vias 1 -> 0
- net SCL: track 74.2 -> 0.00 mm, vias 1 -> 0
- net +BATT: track 69.3 -> 0.00 mm
- net Net-(U3-Vin+): track 61.0 -> 0.00 mm, vias 1 -> 0
- net Net-(A1-A1): track 56.1 -> 0.00 mm, vias 1 -> 0
- net Net-(D10-K): track 55.0 -> 0.00 mm, vias 1 -> 0
- net Net-(A1-D2): track 52.1 -> 0.00 mm, vias 1 -> 0
- net DRV: track 40.8 -> 0.00 mm
- net Net-(A1-A3): track 38.7 -> 0.00 mm, vias 1 -> 0
- net RTN: track 38.4 -> 0.00 mm
- net Net-(A1-A2): track 32.8 -> 0.00 mm, vias 1 -> 0
- net Net-(A1-VIN): track 18.0 -> 0.00 mm, vias 1 -> 0
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- removed copper zone on B.Cu, net GNDPWR
Other:
- board size 81.5 x 76.5 mm -> 1.2 x 1.2 mm

Commit message: Layout
Parts:
- added C12: 0.1u, CAP_BF01:CAP_BF01_AVX, F.Cu at (139.5, 70.5)
- added C13: 47u, Capacitor_THT:CP_Radial_D5.0mm_P2.00mm, F.Cu at (136.0, 75.0)
- TP1: value TestPoint -> V_Buck
- TP10: value TestPoint -> I_Pump
- TP11: value TestPoint -> I_Logic
- TP12: value TestPoint -> PWM
- TP13: value TestPoint -> V_Batt
- TP14: value TestPoint -> TMP
- TP15: value TestPoint -> SCL
- TP16: value TestPoint -> DRV
- TP17: value TestPoint -> RTN
- TP2, TP3: value TestPoint -> GND
- TP4, TP5, TP6: value TestPoint -> PGND
- TP7: value TestPoint -> V_3.3
- TP8: value TestPoint -> V_Esp32
- TP9: value TestPoint -> V_Pump
- moved R14 174.6 mm to (19.0, 39.0)
- moved R12 172.1 mm to (19.0, 34.0)
- moved R13 154.0 mm to (267.3, 125.3)
- moved J-Battery1 131.6 mm to (130.3, 122.2), turned to -90 degrees
- moved S1 126.1 mm to (44.2, 130.8)
- moved S2 126.1 mm to (44.2, 136.9)
- moved S3 126.1 mm to (44.2, 143.1)
- moved C5 118.5 mm to (271.6, 81.7)
- moved CR1 100.3 mm to (281.0, 110.5)
- moved C6 99.6 mm to (273.0, 87.5)
- moved C7 99.6 mm to (273.0, 94.0)
- moved R8 95.7 mm to (204.4, 115.4)
- moved R9 95.7 mm to (204.4, 119.5)
- moved D10 91.1 mm to (140.5, 54.5), turned to 180 degrees
- moved R1 86.4 mm to (32.9, 97.9)
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Routing:
- net Net-(J-Battery1-Pad1): track 0.00 -> 10.4 mm
- net Net-(U1-Vbus): track 0.00 -> 9.09 mm
- net Net-(U1-Vin+): track 0.00 -> 4.60 mm
- net Vdrive: track 0.00 -> 3.42 mm

Commit message: 3/13
Parts:
- added C14: 10n, CAP_BF01:CAP_BF01_AVX, F.Cu at (136.0, 53.0)
- added R17: 9.1, Resistor_THT:R_Axial_DIN0207_L6.3mm_D2.5mm_P10.16mm_Horizontal, F.Cu at (139.0, 47.5)
- added R18: 9.1, Resistor_THT:R_Axial_DIN0207_L6.3mm_D2.5mm_P10.16mm_Horizontal, F.Cu at (138.9, 53.5)
- moved C5 200.0 mm to (85.0, 153.5)
- moved C6 200.0 mm to (86.4, 159.3)
- moved C7 200.0 mm to (86.4, 165.9)
- moved CR1 200.0 mm to (94.4, 182.3)
- moved D9 200.0 mm to (60.2, 176.0)
- moved R13 200.0 mm to (80.7, 197.2)
- moved U3 143.3 mm to (128.0, 50.0)
- moved C8 134.0 mm to (136.0, 61.5), turned to 90 degrees
- moved R11 127.0 mm to (148.0, 50.5), turned to 180 degrees
- moved R14 124.1 mm to (143.0, 33.9), turned to -90 degrees
- moved R12 120.9 mm to (139.5, 44.2), turned to 90 degrees
- moved U2 108.1 mm to (129.2, 171.2), turned to 180 degrees
- moved TP7 96.0 mm to (163.0, 125.5)
- moved TP12 85.0 mm to (136.0, 170.5)
- moved TP9 79.8 mm to (158.0, 47.0), turned to -90 degrees
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Connections:
- C13 pad 1: Net-(A1-VIN) -> Net-(C13-Pad1)
- J-Battery1 pad 2: Net-(U3-Vin+) -> Net-(C13-Pad1)
- R11 pad 1: Net-(U3-Vin+) -> Net-(C13-Pad1)
- TP8 pad 1: Net-(U3-Vin+) -> Net-(C13-Pad1)
- U3 pad 8: +BATT -> Net-(U3-Vbus)
- U3 pad 9: +BATT -> Net-(U3-Vbus)
Routing:
- net Net-(U1-Vin+): track 4.60 -> 24.9 mm, vias 0 -> 2
- net Net-(U1-Vbus): track 9.09 -> 27.4 mm, vias 0 -> 2
- net GND: track 0.00 -> 6.11 mm, vias 0 -> 2
- net Net-(J-Battery1-Pad1): track 10.4 -> 14.2 mm
- net +3.3V: track 0.00 -> 2.71 mm, vias 0 -> 1
