File: MainPCB/MAIN_PCB.kicad_pcb (KiCad board)
At the start: 2 copper layers, 1.2 x 1.2 mm, 72 parts, among them U1 INA226, U2 DRV8871DDA, U3 INA226, U4 CFSH05-20L TR PBFREE, U5 CFSH05-20L TR PBFREE

Commit message: 3/13
Parts:
- moved TP16 204.8 mm to (232.0, 131.5)
- moved J-Pump1 199.5 mm to (227.2, 128.3), turned to 90 degrees
- moved R13 188.9 mm to (244.5, 103.0), turned to 90 degrees
- moved D9 185.7 mm to (229.5, 99.5), turned to -90 degrees
- moved CR1 169.7 mm to (250.0, 114.5)
- moved C7 164.8 mm to (235.5, 95.5), turned to 90 degrees
- moved C5 164.3 mm to (240.1, 99.5), turned to 180 degrees
- moved C6 156.7 mm to (229.5, 95.5), turned to 90 degrees
- moved D2 147.4 mm to (158.0, 168.4), turned to 90 degrees
- moved D3 140.6 mm to (153.0, 168.5), turned to 90 degrees
- moved S1 138.0 mm to (182.3, 131.8)
- moved S2 138.0 mm to (182.3, 137.9)
- moved S3 138.0 mm to (182.3, 144.1)
- moved D4 133.8 mm to (148.0, 168.4), turned to 90 degrees
- moved TP17 129.9 mm to (235.0, 110.0)
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Routing:
- net SDA: track 0.00 -> 103.8 mm
- net +3.3V: track 2.71 -> 89.2 mm, vias 1 -> 3
- net SCL: track 0.00 -> 84.1 mm, vias 0 -> 1
- net Net-(A1-A1): track 0.00 -> 63.6 mm
- net +BATT: track 0.00 -> 32.9 mm, vias 0 -> 1
- net Net-(C13-Pad1): track 0.00 -> 30.5 mm, vias 0 -> 1
- net Net-(A1-VIN): track 0.00 -> 18.9 mm, vias 0 -> 1
- net Net-(U3-Vin+): track 0.00 -> 16.1 mm, vias 0 -> 1
- net Net-(U3-Vbus): track 0.00 -> 13.4 mm, vias 0 -> 1
- net Net-(D10-K): track 0.00 -> 10.9 mm, vias 0 -> 1
- net GND: track 6.11 -> 13.9 mm, vias 2 -> 4
- net Net-(D1-A): track 0.00 -> 7.36 mm
- net Net-(D2-A): track 0.00 -> 7.24 mm
- net Net-(D3-A): track 0.00 -> 6.74 mm
- net Net-(D7-A): track 0.00 -> 6.62 mm
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
Commit message: Nate
Parts:
- moved CR1 94.5 mm to (173.5, 59.0)
- moved TP16 81.8 mm to (155.0, 104.0)
- moved C5 74.2 mm to (172.3, 69.2)
- moved C6 74.2 mm to (161.7, 65.2)
- moved C7 74.2 mm to (167.7, 65.2)
- moved D9 74.2 mm to (161.7, 69.2)
- moved R13 74.2 mm to (176.7, 72.7)
- moved TP12 74.2 mm to (177.2, 79.7)
- moved TP17 74.2 mm to (167.2, 79.7)
- moved U2 74.2 mm to (170.6, 74.7)
- moved J-Pump1 73.1 mm to (155.7, 113.3)
- moved D1 56.2 mm to (166.9, 128.0), turned to -90 degrees
- moved S2 54.7 mm to (168.5, 85.0)
- moved R7 54.2 mm to (104.3, 127.4)
- moved S3 49.5 mm to (168.5, 96.5)
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Routing:
- net Net-(D1-A): track 7.36 -> 0.00 mm
- net Net-(D2-A): track 7.24 -> 0.00 mm
- net Net-(D3-A): track 6.74 -> 0.00 mm
- net Net-(D7-A): track 6.62 -> 0.00 mm
- net Net-(A1-D3): track 6.32 -> 0.00 mm
- net Net-(A1-D9): track 6.15 -> 0.00 mm
- net Net-(D6-A): track 6.00 -> 0.00 mm
- net Net-(D4-A): track 6.00 -> 0.00 mm
- net Net-(A1-D4): track 5.92 -> 0.00 mm
- net Net-(A1-D8): track 5.75 -> 0.00 mm
- net Net-(A1-D5): track 5.52 -> 0.00 mm
- net Net-(D5-A): track 5.38 -> 0.00 mm
- net Net-(A1-D7): track 5.35 -> 0.00 mm
- net Net-(A1-D6): track 5.12 -> 0.00 mm
- net Net-(A1-A1): track 63.6 -> 64.6 mm
Other:
- board size 1.2 x 1.2 mm -> 82 x 99.5 mm

Commit message: Nate
Parts:
- moved D9 50.0 mm to (211.6, 65.0)
- moved CR1 42.5 mm to (215.0, 50.0)
- moved TP17 34.8 mm to (201.6, 74.0)
- moved R13 34.5 mm to (209.0, 60.5), turned to 0 degrees
- moved TP12 29.9 mm to (206.6, 74.0)
- moved C7 17.1 mm to (174.5, 81.0)
- moved U2 12.6 mm to (170.2, 62.1), turned to -90 degrees
- moved C5 9.46 mm to (179.0, 75.9), turned to -90 degrees
- moved S1 5.52 mm to (163.0, 91.3)
- moved S2 5.52 mm to (163.0, 85.5)
- moved S3 5.52 mm to (163.0, 97.0)
- moved C6 4.42 mm to (160.5, 69.5), turned to 0 degrees

Commit message: Almost done
Parts:
- moved CR1 85.7 mm to (152.0, 108.0), turned to -90 degrees
- moved S2 51.9 mm to (150.2, 135.8), turned to -90 degrees
- moved S3 48.4 mm to (134.0, 135.8), turned to -90 degrees
- moved TP17 46.2 mm to (163.7, 100.5)
- moved S1 44.5 mm to (166.8, 135.7), turned to -90 degrees
- moved D9 42.6 mm to (170.7, 77.0), turned to 90 degrees
- moved R13 38.4 mm to (179.0, 84.5), turned to -90 degrees
- moved TP12 35.4 mm to (175.5, 91.0)
- moved U2 30.7 mm to (167.7, 92.7), turned to 180 degrees
- moved C5 13.1 mm to (169.7, 85.2), turned to 180 degrees
- moved TP16 12.3 mm to (160.5, 115.0)
- moved C7 9.81 mm to (164.7, 80.7), turned to 0 degrees
- moved C6 7.02 mm to (164.7, 75.2), turned to 180 degrees
- moved TP9 1.93 mm to (149.0, 68.0)
- moved R10 0.26 mm to (153.0, 69.4)
Routing:
- net PWM: track 0.00 -> 59.2 mm
- net DRV: track 0.00 -> 44.3 mm
- net GND: track 13.9 -> 43.2 mm, vias 4 -> 10
- net GNDPWR: track 3.20 -> 24.6 mm
- net RTN: track 0.00 -> 17.7 mm
- net Vdrive: track 3.42 -> 16.1 mm
- net Net-(U2-ILIM): track 0.00 -> 11.1 mm
- net Net-(J-Battery1-Pad1): track 14.2 -> 12.3 mm
- net (no net): vias 0 -> 21
- added copper zone on F.Cu, net GND
- added copper zone on F.Cu, net GNDPWR

Commit message: Done
Parts:
- added G***: LOGO, LOGO.preety:P16logo, F.Cu at (108.5, 134.0)
- moved TP2 84.2 mm to (176.0, 91.0)
- moved TP5 71.4 mm to (162.5, 59.5)
- moved TP6 65.1 mm to (159.5, 88.0)
- moved TP4 46.1 mm to (132.5, 51.5)
- moved D7 34.6 mm to (168.0, 135.0)
- moved R7 33.7 mm to (138.0, 127.4)
- moved TP12 27.6 mm to (157.0, 111.5)
- moved R6 26.1 mm to (134.5, 127.4)
- moved D6 24.5 mm to (163.0, 135.0)
- moved D2 19.8 mm to (143.0, 135.2)
- moved R5 18.5 mm to (131.0, 127.4)
- moved TP3 15.2 mm to (105.0, 85.0)
- moved D5 14.7 mm to (158.0, 135.0)
- moved TP16 14.6 mm to (158.5, 100.5)
- moved S3 11.7 mm to (143.8, 129.2)
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Connections:
- J-Battery1 pad 3: GND -> GNDPWR
- J-Battery1 pad 4: GNDPWR -> GND
Routing:
- net Net-(D1-A): track 0.00 -> 59.7 mm
- net Net-(A1-A2): track 0.00 -> 57.5 mm, vias 0 -> 1
- net Net-(D7-A): track 0.00 -> 50.9 mm
- net +3.3V: track 89.2 -> 44.8 mm
- net Net-(A1-A3): track 0.00 -> 44.4 mm, vias 0 -> 1
- net Net-(D6-A): track 0.00 -> 42.0 mm
- net Net-(D5-A): track 0.00 -> 33.2 mm
- net Net-(A1-D2): track 0.00 -> 32.8 mm, vias 0 -> 1
- net Net-(D4-A): track 0.00 -> 24.3 mm
- net Net-(D3-A): track 0.00 -> 15.4 mm
- net GND: track 43.2 -> 50.8 mm, vias 10 -> 73
- net Vdrive: track 16.1 -> 23.6 mm
- net PWM: track 59.2 -> 64.9 mm
- net Net-(D2-A): track 0.00 -> 5.08 mm
- net Net-(A1-D9): track 0.00 -> 4.91 mm
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- added copper zone on B.Cu, net +3.3V
- added copper zone on B.Cu, net Vdrive
Other:
- board size 82 x 99.5 mm -> 82 x 96.5 mm
- board text added: "HUMAN COOLER"

Commit message: TMP
Parts:
- moved C8 0.94 mm to (116.3, 68.5)
- moved C13 0.72 mm to (141.0, 69.4)
- moved D1 0.46 mm to (173.0, 134.5)
- moved D5 0.46 mm to (158.0, 134.5)
- moved D6 0.46 mm to (163.0, 134.5)
- moved D7 0.46 mm to (168.0, 134.5)
- moved D2 0.46 mm to (143.0, 134.8)
- moved D3 0.46 mm to (148.0, 134.8)
- moved D4 0.46 mm to (153.0, 134.8)
Routing:
- net +3.3V: track 44.8 -> 87.7 mm
- net Vdrive: track 23.6 -> 14.9 mm
- net Net-(D1-A): track 59.7 -> 61.9 mm
- net Net-(D7-A): track 50.9 -> 52.6 mm
- net Net-(D6-A): track 42.0 -> 43.3 mm
- net Net-(D5-A): track 33.2 -> 34.0 mm
- net GND: track 50.8 -> 51.3 mm, vias 73 -> 74
- net GNDPWR: vias 23 -> 29
- added copper zone on B.Cu, net GND
- added copper zone on B.Cu, net GNDPWR
- added copper zone on F.Cu, net Vdrive
- removed copper zone on B.Cu, net +3.3V
- removed copper zone on B.Cu, net Vdrive
Other:
- board size 82 x 96.5 mm -> 82 x 99.5 mm

Commit message: nate
Parts:
- moved G*** 1.50 mm to (110.0, 134.0)
Routing:
- net GND: track 51.3 -> 50.2 mm
Other:
- board text added: "Nate Muttera"
Changed lines of the file:
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@@
 	(footprint "LOGO.preety:P16logo"
 		(layer "F.Cu")
-		(at 108.5 134)
+		(at 110 134)
 		(property "Reference" "G***"
 			(at 0 0 0)
@@
 			(effects
 				(font
-					(size 1.5 1.5)
+					(size 1.5 10)
 					(thickness 0.3)
 				)
@@
 			(effects
 				(font
-					(size 1.5 1.5)
+					(size 1.5 10)
 					(thickness 0.3)
 				)
@@
 			(effects
 				(font
-					(size 1.27 1.27)
+					(size 1.27 10)
 					(thickness 0.15)
 				)
@@
 			(effects
 				(font
-					(size 1.27 1.27)
+					(size 1.27 10)
 					(thickness 0.15)
 				)
@@
 		(layer "Edge.Cuts")
 	)
+	(gr_text "Nate Muttera"
+		(at 106.5 145.5 0)
+		(layer "F.Cu")
+		(effects
+			(font
+				(size 1.5 1.5)
+				(thickness 0.3)
+				(bold yes)
+			)
+			(justify left bottom)
+		)
+	)
 	(gr_text "HUMAN COOLER"
 		(at 175.5 51.5 270)
@@
 	)
 	(segment
-		(start 143.94 92.44)
-		(end 144.5 93)
+		(start 109.72 78.64)
+		(end 107.5 76.42)
 		(width 0.3)
 		(layer "F.Cu")
@@
 	)
 	(segment
-		(start 106.08 75)
-		(end 106.08 73.58)
+		(start 143.94 92.44)
+		(end 144.5 93)
 		(width 0.3)
 		(layer "F.Cu")
@@
 	)
 	(segment
-		(start 109.72 78.64)
-		(end 106.08 75)
+		(start 136.52 91.44)
+		(end 134.72 91.44)
 		(width 0.3)
 		(layer "F.Cu")
@@
 	)
 	(segment
-		(start 106.08 73.58)
-		(end 108.22 71.44)
+		(start 107.5 76.42)
+		(end 107.5 72.16)
 		(width 0.3)
 		(layer "F.Cu")
@@
 	)
 	(segment
-		(start 136.52 91.44)
-		(end 134.72 91.44)
+		(start 110.923496 71.44)
+		(end 111.622 72.138504)
 		(width 0.3)
 		(layer "F.Cu")
@@
 	)
 	(segment
-		(start 110.923496 71.44)
-		(end 111.622 72.138504)
+		(start 111.622 73.008466)
+		(end 111.22 73.410466)
 		(width 0.3)
 		(layer "F.Cu")
@@
 	)
 	(segment
-		(start 111.622 73.008466)
-		(end 111.22 73.410466)
+		(start 107.5 72.16)
+		(end 108.22 71.44)
 		(width 0.3)
 		(layer "F.Cu")
@@
 	)
 	(segment
+		(start 162.004 91.496)
+		(end 161.435 92.065)
+		(width 0.5)
+		(layer "F.Cu")
+		(net 17)
+	)
+	(segment
 		(start 152 93.5)
 		(end 152 94)
@@
 	)
 	(segment
+		(start 164.206 91.496)
+		(end 162.004 91.496)
+		(width 0.5)
+		(layer "F.Cu")
+		(net 17)
+	)
+	(segment
 		(start 153.5 95.5)
 		(end 155.5 95.5)
@@
 	)
 	(segment
-		(start 152 94)
-		(end 153.5 95.5)
-		(width 1.5)
+		(start 164.775 92.065)
+		(end 164.206 91.496)
+		(width 0.5)
 		(layer "F.Cu")
 		(net 17)
 	)
 	(segment
-		(start 164.775 92.065)
-		(end 161.435 92.065)
-		(width 0.5)
+		(start 152 94)
+		(end 153.5 95.5)
+		(width 1.5)
 		(layer "F.Cu")
 		(net 17)
@@
 	)
 	(segment
-		(start 119.22 74.98)
+		(start 112.26 77.98)
 		(end 116.22 77.98)
 		(width 1.1)
@@
 	)
 	(segment
-		(start 119.22 73.94)
-		(end 119.22 74.98)
+		(start 119.22 74.98)
+		(end 116.22 77.98)
 		(width 1.1)
 		(layer "B.Cu")
@@
 	)
 	(segment
-		(start 112.26 77.98)
-		(end 116.22 77.98)
+		(start 119.22 73.94)
+		(end 119.22 74.98)
 		(width 1.1)
 		(layer "B.Cu")
@@
 	(segment
 		(start 110.771 72.491)
-		(end 114.271 72.491)
+		(end 111.18 72.9)
 		(width 1.1)
 		(layer "B.Cu")
@@
 	)
 	(segment
-		(start 114.68 72.9)
+		(start 111.18 72.9)
 		(end 116.22 72.9)
 		(width 1.1)
@@
 		(width 1.1)
 		(layer "B.Cu")
-		(net 50)
-	)
-	(segment
-		(start 114.271 72.491)
-		(end 114.68 72.9)
-		(width 1.1)
-		(layer "B.Cu")
