File: nolanPCB_Design/nolanPCB_Design.kicad_sch (KiCad schematic)
At the start: 43 parts, among them J1 Pump Bulkhead, J2 TMP Bulkhead, J3 Battery Bulkhead, SW1 Power Switch, SW2 SW_Push, SW3 SW_Push, SW4 SW_Push, SW5 SW_Push, U1 Current Sensor, U2 Motor Driver

Commit message: not sure what was here
Connections:
- net at J1.1, J1.2: now also D1.1 (K); no longer D1.2 (A)
- net at U2.6 (OUT1): now also D1.2 (A); no longer D1.1 (K)
Changed lines of the file:
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@@
 		(lib_id "Device:D_Schottky")
 		(at 246.38 53.34 0)
+		(mirror y)
 		(unit 1)
 		(exclude_from_sim no)
@@
 		(on_board yes)
 		(dnp no)
-		(fields_autoplaced yes)
 		(property "Reference" "D1"
-			(at 246.0625 46.99 0)
+			(at 246.6975 46.99 0)
 			(effects
 				(font
@@
 		)
 		(property "Value" "D_Schottky"
-			(at 246.0625 49.53 0)
+			(at 246.6975 49.53 0)
 			(effects
 				(font
