File: MainPCB_REV2/MAIN_PCB.kicad_sch (KiCad schematic)
At the start: 74 parts, among them U1 INA226, U2 DRV8871DDA, U3 INA226, U4 CFSH05-20L TR PBFREE, U5 CFSH05-20L TR PBFREE

Commit message: 3/23
Parts:
- removed J-Battery1, J-Pump1, J-TMP117: 861-004-213R00Y, 861.preety:861-004-213R00Y, symbol SS-12800-009:SS-12800-009
- removed U4, U5: CFSH05-20L TR PBFREE, symbol 2026-03-11_05-59-29:CFSH05-20L_TR_PBFREE
- added J1: 12V DC PUMP, S4B_PH_SM4_TB:JST_S4B-PH-SM4-TB, symbol S4B-PH-SM4-TB:S4B-PH-SM4-TB
- added J2: 12.8V LFP BATTERY, S4B_PH_SM4_TB:JST_S4B-PH-SM4-TB, symbol S4B-PH-SM4-TB:S4B-PH-SM4-TB
- added J3: TMP117s, S4B_PH_SM4_TB:JST_S4B-PH-SM4-TB, symbol S4B-PH-SM4-TB:S4B-PH-SM4-TB
- C14, C9: footprint CAP_BF01:CAP_BF01_AVX -> Capacitor_THT:C_Rect_L11.0mm_W4.2mm_P10.00mm_MKT
- S1: value TL3315NF250Q -> + BUTTON; footprint TL3315NF250Q:SW_TL3315NF250Q -> B3F_1000:SW_B3F-1000
- S2: value TL3315NF250Q -> - BUTTON; footprint TL3315NF250Q:SW_TL3315NF250Q -> B3F_1000:SW_B3F-1000
- S3: value TL3315NF250Q -> AUTO BUTTON; footprint TL3315NF250Q:SW_TL3315NF250Q -> B3F_1000:SW_B3F-1000
- renumbered U3 to INA226_LOGIC1, U1 to INA226_PUMP1
Connections:
- net +3.3V: now also J3.3
- net GND: now also J2.4, J3.4
- net GNDPWR: now also J1.3, J1.4, J2.3
- net SCL: now also J3.1
- net SDA: now also J3.2
- net at R10.1, R16.2, TP9.1: now also J2.1
- net at C13.1, R11.1, R17.2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: now also J2.2
- net +BATT: no longer names the net of D10.2 (A), R11.2, R14.1, R18.2
- net DRV: no longer names the net of CR1.1, TP16.1, U2.6 (OUT1)
- net DRV: now also J1.1
- net RTN: no longer names the net of TP17.1, U2.8 (OUT2)
- net RTN: now also J1.2
- net Vdrive: no longer names the net of C5.2, C6.1, C7.1, D9.1 (K), R10.2, R15.2, U2.5 (VM)
Other:
- moved on the sheet: A1, C1, C10, C11, C12, C13, C14, C2, C4, C5, C6, C7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

Commit message: a
Parts:
- C14: value 10n -> 0.1uF
- C9: value 10n -> 1uF
- R13: value 32k -> 15k
- R15, R16, R17, R18: value 9.1 -> 8.06
- R8, R9: value 2.2k -> 4.7k
Changed lines of the file:
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@@
 			)
 		)
-		(property "Value" "9.1"
+		(property "Value" "8.06"
 			(at 73.66 102.87 90)
 			(effects
@@
 			)
 		)
-		(property "Value" "9.1"
+		(property "Value" "8.06"
 			(at 109.22 64.77 90)
 			(effects
@@
 			)
 		)
-		(property "Value" "10n"
+		(property "Value" "1uF"
 			(at 57.658 106.68 0)
 			(effects
@@
 			)
 		)
-		(property "Value" "32k"
+		(property "Value" "15k"
 			(at 69.85 154.94 90)
 			(effects
@@
 			)
 		)
-		(property "Value" "9.1"
+		(property "Value" "8.06"
 			(at 111.76 64.77 90)
 			(effects
@@
 			)
 		)
-		(property "Value" "2.2k"
+		(property "Value" "4.7k"
 			(at 240.03 147.32 90)
 			(effects
@@
 			)
 		)
-		(property "Value" "10n"
+		(property "Value" "0.1uF"
 			(at 113.03 76.962 0)
 			(effects
@@
 			)
 		)
-		(property "Value" "9.1"
+		(property "Value" "8.06"
 			(at 73.66 105.41 90)
 			(effects
@@
 			)
 		)
-		(property "Value" "2.2k"
+		(property "Value" "4.7k"
 			(at 254 144.78 90)
 			(effects
