File: MainPCB_REV_3/MainPCB_REV_3.kicad_sch (KiCad schematic)
At the start: 0 parts

Commit message: REV3
Parts:
- added A1: Arduino_Nano_ESP32, Module:Arduino_Nano, symbol MCU_Module:Arduino_Nano_ESP32
- added C1: 10uF, Capacitor_THT:CP_Radial_D5.0mm_P2.00mm, symbol Device:C
- added C10, C11: 100p, CAP_BF01:CAP_BF01_AVX, symbol Device:C
- added C12, C5: 0.1u, CAP_BF01:CAP_BF01_AVX, symbol Device:C
- added C13: 47u, Capacitor_THT:CP_Radial_D5.0mm_P2.00mm, symbol Device:C
- added C14, C9: 10n, Capacitor_THT:C_Rect_L11.0mm_W4.2mm_P10.00mm_MKT, symbol Device:C
- added C2, C4: BQ014E0473J, CAP_BF01:CAP_BF01_AVX, symbol CAP_BF01:BQ014E0473J
- added C3, C8: 0.1uF, CAP_BF01:CAP_BF01_AVX, symbol Device:C
- added C6: 100u, Capacitor_THT:CP_Radial_D5.0mm_P2.00mm, symbol Device:C
- added C7: 10u, Capacitor_THT:CP_Radial_D5.0mm_P2.00mm, symbol Device:C
- added CR1: SA15CA, DO-204AC_SA:DO-204AC_SA, symbol 2026-03-08_02-43-44:SA15CA
- added D1: LED Auto, LED_THT:LED_Oval_W5.2mm_H3.8mm, symbol Device:LED
- added D10: 1N4148, Diode_THT:D_DO-35_SOD27_P7.62mm_Horizontal, symbol Diode:1N4148
- added D11, D8: 1N5817, Diode_THT:D_DO-41_SOD81_P10.16mm_Horizontal, symbol Diode:1N5817
- added D2: BAT3, LED_THT:LED_Oval_W5.2mm_H3.8mm, symbol Device:LED
- added D3: BAT2, LED_THT:LED_Oval_W5.2mm_H3.8mm, symbol Device:LED
- added D4: BAT1, LED_THT:LED_Oval_W5.2mm_H3.8mm, symbol Device:LED
- added D5: MAN 3, LED_THT:LED_Oval_W5.2mm_H3.8mm, symbol Device:LED
- added D6: MAN 2, LED_THT:LED_Oval_W5.2mm_H3.8mm, symbol Device:LED
- added D7: MAN 1, LED_THT:LED_Oval_W5.2mm_H3.8mm, symbol Device:LED
- added D9: 80SQ045NRLG, 80SQ045NRLG:DIOAD2860W130L840D505, symbol 80SQ045NRLG:80SQ045NRLG
- added INA226_LOGIC1, INA226_PUMP1: INA226, Package_SO:VSSOP-10_3x3mm_P0.5mm, symbol Sensor_Energy:INA226
- added J1: 12V DC PUMP, S4B_PH_SM4_TB:JST_S4B-PH-SM4-TB, symbol S4B-PH-SM4-TB:S4B-PH-SM4-TB
- added J2: 12.8V LFP BATTERY, S4B_PH_SM4_TB:JST_S4B-PH-SM4-TB, symbol S4B-PH-SM4-TB:S4B-PH-SM4-TB
- added J3: TMP117s, S4B_PH_SM4_TB:JST_S4B-PH-SM4-TB, symbol S4B-PH-SM4-TB:S4B-PH-SM4-TB
- added L2: LQH44PH220MPRL, IND_LQH44PN:IND_LQH44PN_PR_MUR, symbol IND_LQH44PN:LQH44PH220MPRL
- added R1, R2, R3, R4, R5, R6, R7: 56, Resistor_THT:R_Axial_DIN0207_L6.3mm_D2.5mm_P10.16mm_Horizontal, symbol Device:R
- added R10, R11: Shunt, Resistor_SMD:R_1206_3216Metric, symbol Device:R
- added R12: 100k, Resistor_THT:R_Axial_DIN0207_L6.3mm_D2.5mm_P10.16mm_Horizontal, symbol Device:R
- added R13: 32k, Resistor_THT:R_Axial_DIN0207_L6.3mm_D2.5mm_P10.16mm_Horizontal, symbol Device:R
- added R14: 390k, Resistor_THT:R_Axial_DIN0207_L6.3mm_D2.5mm_P10.16mm_Horizontal, symbol Device:R
- added R15, R16, R17, R18: 9.1, Resistor_THT:R_Axial_DIN0207_L6.3mm_D2.5mm_P10.16mm_Horizontal, symbol Device:R
- added R8, R9: 2.2k, Resistor_THT:R_Axial_DIN0207_L6.3mm_D2.5mm_P10.16mm_Horizontal, symbol Device:R
- added S1: + BUTTON, B3F_1000:SW_B3F-1000, symbol TL3315NF250Q:TL3315NF250Q
- added S2: - BUTTON, B3F_1000:SW_B3F-1000, symbol TL3315NF250Q:TL3315NF250Q
- added S3: AUTO BUTTON, B3F_1000:SW_B3F-1000, symbol TL3315NF250Q:TL3315NF250Q
- added TP1: V_Buck, TestPoint:TestPoint_THTPad_D1.5mm_Drill0.7mm, symbol Connector:TestPoint
- added TP10: I_Pump, TestPoint:TestPoint_THTPad_D1.5mm_Drill0.7mm, symbol Connector:TestPoint
- added TP11: I_Logic, TestPoint:TestPoint_THTPad_D1.5mm_Drill0.7mm, symbol Connector:TestPoint
- added TP12: PWM, TestPoint:TestPoint_THTPad_D1.5mm_Drill0.7mm, symbol Connector:TestPoint
- added TP13: V_Batt, TestPoint:TestPoint_THTPad_D1.5mm_Drill0.7mm, symbol Connector:TestPoint
- added TP14: TMP, TestPoint:TestPoint_THTPad_D1.5mm_Drill0.7mm, symbol Connector:TestPoint
- added TP15: SCL, TestPoint:TestPoint_THTPad_D1.5mm_Drill0.7mm, symbol Connector:TestPoint
- added TP16: DRV, TestPoint:TestPoint_THTPad_D1.5mm_Drill0.7mm, symbol Connector:TestPoint
- added TP17: RTN, TestPoint:TestPoint_THTPad_D1.5mm_Drill0.7mm, symbol Connector:TestPoint
- added TP2, TP3: GND, TestPoint:TestPoint_THTPad_D1.5mm_Drill0.7mm, symbol Connector:TestPoint
- added TP4, TP5, TP6: PGND, TestPoint:TestPoint_THTPad_D1.5mm_Drill0.7mm, symbol Connector:TestPoint
- added TP7: V_3.3, TestPoint:TestPoint_THTPad_D1.5mm_Drill0.7mm, symbol Connector:TestPoint
- added TP8: V_Esp32, TestPoint:TestPoint_THTPad_D1.5mm_Drill0.7mm, symbol Connector:TestPoint
- added TP9: V_Pump, TestPoint:TestPoint_THTPad_D1.5mm_Drill0.7mm, symbol Connector:TestPoint
- added U2: DRV8871DDA, Package_SO:Texas_HTSOP-8-1EP_3.9x4.9mm_P1.27mm_EP2.95x4.9mm_Mask2.4x3.1mm_ThermalVias, symbol Driver_Motor:DRV8871DDA
Connections:
- new net: CR1.1, J1.1, TP16.1, U2.6 (OUT1)
- new net: J1.2, TP17.1, U2.8 (OUT2)
- new net: C11.1, C9.2, D11.1 (K), INA226_PUMP1.10 (Vin+), R16.1
- new net: J2.1, R10.1, R16.2, TP9.1
- new net: C14.2, INA226_LOGIC1.10 (Vin+), R17.1
- new net: C13.1, J2.2, R11.1, R17.2, TP8.1
- new net: D2.2 (A), R7.2
- new net: D7.2 (A), R2.2
- new net: A1.12 (D9), R7.1
- new net: D6.2 (A), R3.2
- new net: A1.20 (A1), R12.1, R14.2, TP13.1
- new net: A1.7 (D4), R2.1
- new net: C10.2, C9.1, D8.1 (K), INA226_PUMP1.8 (Vbus), INA226_PUMP1.9 (Vin-), R15.1
- new net: D3.2 (A), R6.2
- new net: A1.30 (VIN), C12.2, C2.1, L2.2, TP1.1
- new net: R13.1, U2.4 (ILIM)
- new net: C5.2, C6.1, C7.1, D9.1 (K), R10.2, R15.2, U2.5 (VM)
- new net: C14.1, INA226_LOGIC1.8 (Vbus), INA226_LOGIC1.9 (Vin-), R18.1
- new net: A1.22 (A3), S2.1, S2.2
- new net: A1.10 (D7), R5.1
- new net: A1.11 (D8), R6.1
- new net: A1.21 (A2), S1.1, S1.2
- new net: A1.5 (D2), S3.3, S3.4
- new net: A1.6 (D3), R1.1
- new net: A1.8 (D5), R3.1
- new net: A1.9 (D6), R4.1
- new net: D10.2 (A), R11.2, R14.1, R18.2
- new net: D1.2 (A), R1.2
- new net: D4.2 (A), R5.2
- new net: C4.1, D10.1 (K), L2.1
- new net: D5.2 (A), R4.2
- new net +3.3V: A1.17 (3V3), C1.1, C3.2, C8.2, INA226_LOGIC1.2 (A0), INA226_LOGIC1.6 (VS), INA226_PUMP1.6 (VS), J3.3, R8.2, R9.2, TP7.1
- new net GND: A1.29 (GND), A1.4 (GND), C1.2, C12.1, C13.2, C2.2, C3.1, C4.2, C5.1, C7.2, C8.1, D1.1 (K), D2.1 (K), D3.1 (K), D4.1 (K), D5.1 (K), D6.1 (K), D7.1 (K), INA226_LOGIC1.1 (A1), INA226_LOGIC1.7 (GND), INA226_PUMP1.1 (A1), INA226_PUMP1.2 (A0), INA226_PUMP1.7 (GND), J2.4, J3.4, R12.2, R13.2, S1.3, S1.4, S2.3, S2.4, S3.1, S3.2, TP2.1, TP3.1, U2.1 (GND), U2.2 (IN2), U2.9 (GND)
- new net GNDPWR: C10.1, C11.2, C6.2, CR1.2, D11.2 (A), D8.2 (A), D9.2 (A), J1.3, J1.4, J2.3, TP4.1, TP5.1, TP6.1, U2.7 (PWRGND)
- new net PWM: A1.19 (A0), TP12.1, U2.3 (IN1)
- new net SCL: A1.24 (SCL/A5), INA226_LOGIC1.5 (SCL), INA226_PUMP1.5 (SCL), J3.1, R9.1, TP15.1
- new net SDA: A1.23 (SDA/A4), INA226_LOGIC1.4 (SDA), INA226_PUMP1.4 (SDA), J3.2, R8.1, TP10.1, TP11.1, TP14.1
- no-connect marks 0 -> 9

Commit message: NORA
Parts:
- removed R12: 100k, Resistor_THT:R_Axial_DIN0207_L6.3mm_D2.5mm_P10.16mm_Horizontal, symbol Device:R
- removed R14: 390k, Resistor_THT:R_Axial_DIN0207_L6.3mm_D2.5mm_P10.16mm_Horizontal, symbol Device:R
- added D12: 1N5817, Diode_THT:D_DO-41_SOD81_P10.16mm_Horizontal, symbol Diode:1N5817
- added IC1: NORA-W106-10B, NORAW10610B, symbol NORA-W106-10B:NORA-W106-10B
- R13: value 32k -> 14k
- R8, R9: value 2.2k -> 4.7k
Connections:
- net GND: now also D12.2 (A)
- net at TP13.1: now also R11.2, R18.2; no longer A1.20 (A1)
- new net: D10.2 (A), D12.1 (K)
- no-connect marks 9 -> 14
Other:
- moved on the sheet: A1, C1, C12, C2, C4, D1, D10, D2, D3, D4, D5, D6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
