File: MainPCB_REV_3/MainPCB_REV_3.kicad_sch (KiCad schematic)
At the start: 72 parts, among them IC1 NORA-W106-10B, J1 12V DC PUMP, J2 12.8V LFP BATTERY, J3 TMP117s, U2 DRV8871DDA

Commit message: nate
Parts:
- removed C1: 10uF, Capacitor_THT:CP_Radial_D5.0mm_P2.00mm, symbol Device:C
- removed C10, C11: 100p, CAP_BF01:CAP_BF01_AVX, symbol Device:C
- removed C12, C5: 0.1u, CAP_BF01:CAP_BF01_AVX, symbol Device:C
- removed C14, C9: 10n, Capacitor_THT:C_Rect_L11.0mm_W4.2mm_P10.00mm_MKT, symbol Device:C
- removed C2, C4: BQ014E0473J, CAP_BF01:CAP_BF01_AVX, symbol CAP_BF01:BQ014E0473J
- removed C3, C8: 0.1uF, CAP_BF01:CAP_BF01_AVX, symbol Device:C
- removed C7: 10u, Capacitor_THT:CP_Radial_D5.0mm_P2.00mm, symbol Device:C
- removed CR1: SA15CA, DO-204AC_SA:DO-204AC_SA, symbol 2026-03-08_02-43-44:SA15CA
- removed D1: LED Auto, LED_THT:LED_Oval_W5.2mm_H3.8mm, symbol Device:LED
- removed D10: 1N4148, Diode_THT:D_DO-35_SOD27_P7.62mm_Horizontal, symbol Diode:1N4148
- removed D11, D12, D8: 1N5817, Diode_THT:D_DO-41_SOD81_P10.16mm_Horizontal, symbol Diode:1N5817
- removed D2: BAT3, LED_THT:LED_Oval_W5.2mm_H3.8mm, symbol Device:LED
- removed D3: BAT2, LED_THT:LED_Oval_W5.2mm_H3.8mm, symbol Device:LED
- removed D4: BAT1, LED_THT:LED_Oval_W5.2mm_H3.8mm, symbol Device:LED
- removed D5: MAN 3, LED_THT:LED_Oval_W5.2mm_H3.8mm, symbol Device:LED
- removed D6: MAN 2, LED_THT:LED_Oval_W5.2mm_H3.8mm, symbol Device:LED
- removed D7: MAN 1, LED_THT:LED_Oval_W5.2mm_H3.8mm, symbol Device:LED
- removed D9: 80SQ045NRLG, 80SQ045NRLG:DIOAD2860W130L840D505, symbol 80SQ045NRLG:80SQ045NRLG
- removed IC1: NORA-W106-10B, NORAW10610B, symbol NORA-W106-10B:NORA-W106-10B
- removed J2: 12.8V LFP BATTERY, S4B_PH_SM4_TB:JST_S4B-PH-SM4-TB, symbol S4B-PH-SM4-TB:S4B-PH-SM4-TB
- removed R1, R2, R3, R4, R5, R6, R7: 56, Resistor_THT:R_Axial_DIN0207_L6.3mm_D2.5mm_P10.16mm_Horizontal, symbol Device:R
- removed R10, R11: Shunt, Resistor_SMD:R_1206_3216Metric, symbol Device:R
- removed R13: 14k, Resistor_THT:R_Axial_DIN0207_L6.3mm_D2.5mm_P10.16mm_Horizontal, symbol Device:R
- removed R15, R16, R17, R18: 9.1, Resistor_THT:R_Axial_DIN0207_L6.3mm_D2.5mm_P10.16mm_Horizontal, symbol Device:R
- removed R8, R9: 4.7k, Resistor_THT:R_Axial_DIN0207_L6.3mm_D2.5mm_P10.16mm_Horizontal, symbol Device:R
- removed TP13: V_Batt, TestPoint:TestPoint_THTPad_D1.5mm_Drill0.7mm, symbol Connector:TestPoint
- removed TP6: PGND, TestPoint:TestPoint_THTPad_D1.5mm_Drill0.7mm, symbol Connector:TestPoint
- added C1, C6: 10uF, PCM_JLCPCB:C_1206, symbol PCM_JLCPCB-Capacitors:1206,10uF
- added C10, C8: 470nF, PCM_JLCPCB:C_0805, symbol PCM_JLCPCB-Capacitors:0805,470nF
- added C11, C2, C7, C9: 100nF, PCM_JLCPCB:C_1206, symbol PCM_JLCPCB-Capacitors:1206,100nF
- added C3, C4: 220nF, PCM_JLCPCB:C_1206, symbol PCM_JLCPCB-Capacitors:1206,220nF
- added D1, D10, D9: DSL34, PCM_JLCPCB:D_SOD-123FL, symbol PCM_JLCPCB-Diodes:Schottky,DSL34
- added D2, D3, D8: Red, PCM_JLCPCB:D_0805, symbol PCM_JLCPCB-Diodes:LED,0805,Red
- added D4, D5: Yellow, PCM_JLCPCB:D_0805, symbol PCM_JLCPCB-Diodes:LED,0805,Yellow
- added D6, D7: Green, PCM_JLCPCB:D_0805, symbol PCM_JLCPCB-Diodes:LED,0805,Green
- added F1: Fuse, fuse:FUSE_658_LTF, symbol Device:Fuse
- added J2: Barrel_Jack, Connector_BarrelJack:BarrelJack_CUI_PJ-079BH_Horizontal, symbol Connector:Barrel_Jack
- added R1, R2: 4.7kΩ, PCM_JLCPCB:R_1206, symbol PCM_JLCPCB-Resistors:1206,4.7kΩ
- added R10: 15kΩ, PCM_JLCPCB:R_0805, symbol PCM_JLCPCB-Resistors:0805,15kΩ
- added R11, R12, R14, R15: 8.2Ω, PCM_JLCPCB:R_1206, symbol PCM_JLCPCB-Resistors:1206,10Ω
- added R13, R16: 10mΩ, PCM_JLCPCB:R_1206, symbol PCM_JLCPCB-Resistors:1206,100mΩ
- added R3, R4, R5, R6, R7, R8, R9: 56Ω, PCM_JLCPCB:R_0805, symbol PCM_JLCPCB-Resistors:0805,56Ω
- added SW1: L101011MS02Q, switch:SW_1MS02Q_CNK, symbol 2026-04-24_06-13-35:L101011MS02Q
- S1, S2, S3: footprint B3F_1000:SW_B3F-1000 -> TL3315NF250Q:SW_TL3315NF250Q
- U1: renamed from INA226_LOGIC1; footprint Package_SO:VSSOP-10_3x3mm_P0.5mm -> Package_SO:TSSOP-10_3x3mm_P0.5mm
- U2: renamed from INA226_PUMP1; footprint Package_SO:VSSOP-10_3x3mm_P0.5mm -> Package_SO:TSSOP-10_3x3mm_P0.5mm
- renumbered C13 to C12, C6 to C5, L2 to L1, TP2 to TP1, TP9 to TP12, TP8 to TP13, TP3 to TP2, TP4 to TP3, TP5 to TP4, TP15 to TP5, TP7 to TP6, TP1 to TP7, TP16 to TP8, TP12 to TP9, U2 to U3
Connections:
- net GNDPWR is gone; now on net GND: C5.2, J1.3, J1.4, TP3.1, TP4.1, U3.7 (PWRGND)
- net +3.3V: now also C1.2, C11.2, C9.2, R1.2, R2.2
- net GND: now also C1.1, C11.1, C2.1, C3.1, C4.1, C6.1, C7.1, C9.1, D10.2, D2.1, D3.1, D4.1, D5.1, D6.1, D7.1, D8.1, D9.2, J2.1, R10.2
- net SCL: now also R2.1
- net SDA: now also R1.1
- net at J1.1, TP8.1, U3.6 (OUT1): now also D9.1
- net at U2.10 (Vin+): now also C8.1, R12.1
- net at TP12.1: now also C12.1, TP13.1, R12.2, R13.1, R15.1, R16.1, SW1.1
- net at U1.10 (Vin+): now also C10.1, R15.2
- net at A1.12 (D9): now also R3.1
- net at A1.7 (D4): now also R8.1
- net at U2.8 (Vbus), U2.9 (Vin-): now also C8.2, R11.1
- net at A1.30 (VIN), L1.2, TP7.1: now also C2.2, C3.2
- net at U3.4 (ILIM): now also R10.1
- net at C5.1, U3.5 (VM): now also C6.2, C7.2, D10.1, R11.2, R13.2
- net at U1.8 (Vbus), U1.9 (Vin-): now also C10.2, R14.1
- net at A1.10 (D7): now also R5.1
- net at A1.11 (D8): now also R4.1
- net at A1.6 (D3): now also R9.1
- net at A1.8 (D5): now also R7.1
- net at A1.9 (D6): now also R6.1
- net at L1.1: now also C4.2, D1.1
- new net: D7.2, R8.2
- new net: D1.2, R14.2, R16.2
- new net: D2.2, R3.2
- new net: F1.2, SW1.2
- new net: F1.1, J2.2
- new net: D4.2, R5.2
- new net: D8.2, R9.2
- new net: D3.2, R4.2
- new net: D5.2, R6.2
- new net: D6.2, R7.2
Other:
- moved on the sheet: A1, L1, S1, S2, S3, TP13, TP5, TP6, TP7

Commit message: Final
Parts:
- removed R13, R16: 10mΩ, PCM_JLCPCB:R_1206, symbol PCM_JLCPCB-Resistors:1206,100mΩ
- added R13, R16: 1Ω, PCM_JLCPCB:R_1206, symbol PCM_JLCPCB-Resistors:1206,1Ω
Connections:
- net at D1.2, R14.2: now also R16.2
- net at C12.1, R12.2, R15.1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: now also R13.2, R16.1
- net at C5.1, C6.2, C7.2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: now also R13.1
- no-connect marks 14 -> 13
