File: MainPCB_REV_3/MainPCB_REV_3.kicad_pcb (KiCad board)
At the start: 2 copper layers, 66 parts, among them J1 12V DC PUMP, J2 Barrel_Jack, J3 TMP117s, SW1 L101011MS02Q, U1 INA226, U2 INA226, U3 DRV8871DDA

Commit message: Final
Parts:
- added G***: LOGO, LOGO.preety:P16logo, F.Cu at (161.5, 70.0)
- C12: value 47u -> 47uF
- L1: value LQH44PH220MPRL -> 22uH
- R13, R16: value 10mΩ -> 1Ω
- moved A1 83.5 mm to (167.7, 121.3), turned to 180 degrees
- moved TP17 82.7 mm to (177.0, 65.8), turned to -90 degrees
- moved TP8 81.8 mm to (172.0, 65.8), turned to 90 degrees
- moved TP14 78.0 mm to (182.0, 75.2), turned to 90 degrees
- moved TP2 77.3 mm to (181.5, 116.5)
- moved J2 70.3 mm to (128.8, 76.0)
- moved TP9 64.1 mm to (139.0, 66.2)
- moved SW1 55.1 mm to (126.0, 109.0), turned to 0 degrees
- moved F1 54.2 mm to (124.5, 90.0), turned to -90 degrees
- moved C2 52.6 mm to (145.5, 121.3)
- moved TP6 52.0 mm to (148.5, 91.8)
- moved S2 49.1 mm to (174.5, 121.9)
- moved TP10 48.7 mm to (148.0, 81.2)
- moved S1 48.5 mm to (174.5, 115.0)
- moved R3 47.9 mm to (172.0, 91.9)
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Connections:
- R13 pad 1: Net-(C12-Pad1) -> Net-(U3-VM)
- R13 pad 2: Net-(U3-VM) -> Net-(C12-Pad1)
Routing:
- net SDA: track 0.00 -> 114.6 mm
- net +3.3V: track 0.00 -> 102.9 mm, vias 0 -> 2
- net SCL: track 0.00 -> 93.9 mm, vias 0 -> 2
- net Net-(U3-OUT1): track 0.00 -> 47.8 mm
- net Net-(U3-OUT2): track 0.00 -> 45.1 mm
- net PWM: track 0.00 -> 40.5 mm
- net Net-(C12-Pad1): track 0.00 -> 40.2 mm
- net Net-(A1-A3): track 0.00 -> 34.1 mm, vias 0 -> 1
- net Net-(A1-D2): track 0.00 -> 30.6 mm, vias 0 -> 1
- net Net-(A1-A2): track 0.00 -> 30.4 mm, vias 0 -> 1
- net GND: track 0.00 -> 19.3 mm, vias 0 -> 67
- net Net-(F1-Pad1): track 0.00 -> 15.8 mm
- net Net-(U2-Vin+): track 0.00 -> 14.0 mm
- net Net-(A1-VIN): track 0.00 -> 12.3 mm
- net Net-(F1-Pad2): track 0.00 -> 11.1 mm
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- added copper zone on B.Cu, net GND
- added copper zone on F.Cu, net GND
- added copper zone on F.Cu, net Net-(U3-VM)
Other:
- board outline added: 70.2 x 67.8 mm
- board text added: "-Nate Muttera"
- board text added: "CRYOBOD"
- board text added: "HUMAN COOLER"
